File: BMS/ECAD/IMD/IMD/IMD_CTRL.kicad_sch (KiCad schematic)
At the start: 36 parts, among them Q14 FDN352AP, Q15 2N7002, Q401 FDN352AP, Q402 FDN352AP, U401 4017, U402 NE555D, U403 NE555D, U404 NE555D, U405 74HC123, U406 74HC74

Commit message: add several subcomponent starts
Parts:
- added unit 3 of U404
- added unit 2 of U404
- added unit 2 of U405
- added unit 3 of U405
- renumbered C405 to C401, C403 to C402, C401 to C403, C406 to C405, C402 to C406, D403 to D402, D404 to D403, D402 to D404, Q14 to Q401, Q401 to Q402, Q15 to Q403, Q402 to Q404, R405 to R401, R406 to R402, R402 to R405, R401 to R406, R411 to R407, R412 to R408, R413 to R409, R407 to R410, R408 to R411, R31 to R412, R410 to R413, R409 to R414, R414 to R415, U403 to U401, U404 to U402, U402 to U403, U406 to U404, U401 to U406
Connections:
- net !TEST_EN: now also U404.8 (~{Q}); no longer U404.8 (~{Q})
- net !TEST_RES: now also U404.13 (~{R}); no longer U404.13 (~{R})
- net CLK_1s2: now also U405.10 (B), U405.9 (A); no longer U405.10 (B), U405.9 (A)
- net CLK_1s2_pulsed: now also U405.5 (Q); no longer U405.5 (Q)
- net NEG_Switch: now also U404.11 (C); no longer U404.11 (C)
- net TEST_Qued: now also U404.12 (D); no longer U404.12 (D)
- net at C408.2: now also U405.6 (Cext); no longer U405.6 (Cext)
- net at R411.2: now also U405.7 (RCext); no longer U405.7 (RCext)
Other:
- moved on the sheet: Q401, Q402, Q403, Q404, R412, R413, R414, R415, U406
