File: BMS/ECAD/HVDCDC/HV_DCDC_Module.kicad_sch (KiCad schematic)
At the start: 96 parts, among them Q1 NMOS, Q2 NMOS, Q3 NMOS, Q4 NMOS, T1 PA2002NL, T2 PA2002NL, T3 Transformer_1P_2S, T4 Transformer_1P_1S, U1 LMV431, U2 CNY17-1, U3 UCC27324, U4 UCC27324

Commit message: DCDC Schematic 80%
Parts:
- added C33: 100nC, symbol Device:C
- added C34, C35, C37, C38, C39: 1uC, symbol Device:C
- added C36: 2.2nC, symbol Device:C
- added C40: 100uC, symbol Device:C_Polarized
- added C41: 100pC, symbol Device:C
- added R31, R32, R39, R40, R44: 10kR, symbol Device:R
- added R33, R34: 17.8kR, symbol Device:R
- added R35: 29.4kR, symbol Device:R
- added R36: 59kR, symbol Device:R
- added R37: 90.9kR, symbol Device:R
- added R38, R42: 1kR, symbol Device:R
- added R41: 2.49kR, symbol Device:R
- added R43: 1.58kR, symbol Device:R
- added U5: ~, symbol HVDCDC_special:UCC28950PW
Connections:
- net +5V_Ref: now also C34.1, R31.1, R36.2, R37.2, R38.2, U5.1 (VREF)
- net GD-_S1: no longer R6.1
- net GNDA: now also C33.2, C34.2, C35.2, C36.2, C38.2, C39.1, C40.2, C41.2, R32.2, R33.2, R34.2, R35.2, R41.1, R43.2, U5.24 (GND)
- net ISens: now also R42.1
- net Switch_S1: now also U5.22 (OUTA)
- net Switch_S2: now also U5.21 (OUTB)
- net Switch_S3: now also U5.20 (OUTC)
- net Switch_S4: now also U5.19 (OUTD)
- net VSens: now also C38.1, R40.2, R41.2
- net at C2.1, C4.1, D2.1 (K)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: now also Q3.1 (D)
- net +10V renamed +12V
- net +12V: now also C39.2, C40.1, U5.23 (VDD)
- new net: R39.1, U5.4 (COMP)
- new net: C37.1, R39.2
- new net: R33.1, U5.6 (DELAB)
- new net: R35.1, U5.9 (TMIN)
- new net: C33.1, R31.2, R32.1, U5.2 (EA+)
- new net: R43.1, R44.2, U5.14 (ADEL)
- new net: C36.1, R38.1, U5.12 (DCM)
- new net: R36.1, U5.10 (RT)
- new net: R37.1, U5.11 (RSUM)
- new net: C41.1, R42.2, R44.1, U5.15 (CS)
- new net: C37.2, R40.1, U5.3 (EA-)
- new net: C35.1, U5.5 (SS/EN)
- new net: R34.1, U5.7 (DELCD)
- new net GD-_S2: R6.1
- no-connect marks 0 -> 4
Other:
- note added: "Control IC"
- note added: "Current Sense"
- note added: "Feedback Circuit"
- note added: "Gate Drive"
- note added: "H-Bridge"
- note added: "HV Indicator Driver als Modul für aux supply mit nachgeschaltetem LDO von 15V auf 12V"
- note added: "Output Filter"
- note added: "Rectifier"
- note added: "ToDO Footprints und konkrete teileauswahl hinsichtlich kosten Einschaltlogik per LVMS (analog zu BR mit keliern Zelle NiCd?!) Auxillary supply mit HVIndicator (Module steckpaltz vorsehen / mit in einschaltlogik / power sequencing aufnehmen Debug LEDS sync line ausbinden fr modul parallelisierung Trafo selbstfertigung planen Eigenes DCDC HV Relais plus precharge (einfach den precharge circuit nehm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"
- note removed: "10-12V DC supply 45mA via HV Indicator schaltung?"
- moved on the sheet: C1, C10, C11, C12, C13, C14, C15, C16, C17, C18, C19, C2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
