File: BMS/ECAD/StackController/Balancing.kicad_sch (KiCad schematic)
At the start: 5 parts

Commit message: finish V09 of stack controller and HV indicator
Parts:
- R18: value 18R -> 39R
Other:
- company: (none) -> Lukas Deeken Elektronik
- title: (none) -> Stack Controller
Changed lines of the file:
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@@
 	(generator_version "9.0")
 	(paper "A4")
+	(title_block
+		(title "Stack Controller")
+		(date "2026-02-27")
+		(rev "1.0")
+		(company "Lukas Deeken Elektronik")
+	)
 	(text_box "Balancing strom geht durch RBal -> RSwitch -> RF\n\nRF = 10Ohm\nRSwitch_min = 1,6Ohm\nRbal = 39Ohm\n\nU_Max_cell = 4,25V\n\nIMax_bal = 4,25V/29,6Ohm = 143,6mA\n\nhalbieren paralleler stromdfluss?"
 		(exclude_from_sim no)
@@
 			)
 		)
-		(property "Value" "18R"
+		(property "Value" "39R"
 			(at 154.432 115.57 90)
 			(effects
@@
 			)
 		)
-		(property "Datasheet" "CRGH2512J47R"
+		(property "Datasheet" ""
 			(at 149.86 116.84 0)
 			(effects

Commit message: started layout BMS slave
Parts:
- renumbered C15 to C28, C16 to C29, C17 to C30, R17 to R39, R18 to R40
