File: BMS/ECAD/StackController/StackController.kicad_pcb (KiCad board)
At the start: 2 copper layers, 85.8 x 62 mm, 209 parts, among them Q1 BC846, Q2 BC846, U1 TLE9012, U2 TMUX1309A, U3 TMUX1309A

Commit message: pack controller close to finished and startet pack controller
Routing:
- net Net-(StackPower1-A): track 3.11 -> 1.66 mm
- net VStack: track 27.8 -> 26.9 mm
- net /Balancing_0/U: track 25.2 -> 25.9 mm
- net Net-(U1-U12P): track 25.6 -> 26.3 mm
