File: BMS/ECAD/StackController/StackController.kicad_pcb (KiCad board)
At the start: 2 copper layers, 85.8 x 62 mm, 209 parts, among them Q1 BC846, Q2 BC846, U1 TLE9012, U2 TMUX1309A, U3 TMUX1309A

Commit message: yes
Parts:
- C1, C2, C3, C4, C5: value 10uC 16V -> 10uC 35V; footprint Capacitor_SMD:C_0603_1608Metric -> Capacitor_SMD:C_0805_2012Metric
- R4: value 170kR 0,1% 25ppm/C -> 162kR 0,1% 25ppm/C
- moved C5 0.55 mm to (55.6, 63.2)
- moved C3 0.36 mm to (51.7, 63.2)
- moved C4 0.15 mm to (53.6, 63.2)
- renumbered Bot_IsoUART1 to Bot_IsoUART, Top_IsoUART1 to Top_IsoUART
Routing:
- net TMP_MUX1: track 61.5 -> 60.8 mm
- net /Balancing_5/U-1: track 95.3 -> 95.9 mm
Other:
- board text removed: "HV"
- board text removed: "LV"
