File: BMS/ECAD/StackController/StackController.kicad_sch (KiCad schematic)
At the start: 126 parts, among them Q1 BC846, Q2 BC846, U1 TLE9012

Commit message: yes
Parts:
- C1, C2, C3, C4, C5: value 10uC 16V -> 10uC 35V; footprint Capacitor_SMD:C_0603_1608Metric -> Capacitor_SMD:C_0805_2012Metric
- R4: value 170kR 0,1% 25ppm/C -> 162kR 0,1% 25ppm/C
Changed lines of the file:
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@@
 			)
 		)
-		(property "Value" "10uC 16V"
+		(property "Value" "10uC 35V"
 			(at 68.834 106.426 0)
 			(hide yes)
@@
 			)
 		)
-		(property "Footprint" "Capacitor_SMD:C_0603_1608Metric"
+		(property "Footprint" "Capacitor_SMD:C_0805_2012Metric"
 			(at 69.5452 107.95 0)
 			(hide yes)
@@
 			)
 		)
-		(property "Value" "10uC 16V"
+		(property "Value" "10uC 35V"
 			(at 53.594 106.426 0)
 			(hide yes)
@@
 			)
 		)
-		(property "Footprint" "Capacitor_SMD:C_0603_1608Metric"
+		(property "Footprint" "Capacitor_SMD:C_0805_2012Metric"
 			(at 54.3052 107.95 0)
 			(hide yes)
@@
 			)
 		)
-		(property "Value" "10uC 16V"
+		(property "Value" "10uC 35V"
 			(at 45.974 106.426 0)
 			(hide yes)
@@
 			)
 		)
-		(property "Footprint" "Capacitor_SMD:C_0603_1608Metric"
+		(property "Footprint" "Capacitor_SMD:C_0805_2012Metric"
 			(at 46.6852 107.95 0)
 			(hide yes)
@@
 			)
 		)
-		(property "Value" "10uC 16V"
+		(property "Value" "10uC 35V"
 			(at 61.214 106.426 0)
 			(hide yes)
@@
 			)
 		)
-		(property "Footprint" "Capacitor_SMD:C_0603_1608Metric"
+		(property "Footprint" "Capacitor_SMD:C_0805_2012Metric"
 			(at 61.9252 107.95 0)
 			(hide yes)
@@
 			)
 		)
-		(property "Value" "10uC 16V"
+		(property "Value" "10uC 35V"
 			(at 78.994 104.14 0)
 			(show_name no)
@@
 			)
 		)
-		(property "Footprint" "Capacitor_SMD:C_0603_1608Metric"
+		(property "Footprint" "Capacitor_SMD:C_0805_2012Metric"
 			(at 77.1652 107.95 0)
 			(hide yes)
@@
 			)
 		)
-		(property "Value" "170kR 0,1% 25ppm/C"
+		(property "Value" "162kR 0,1% 25ppm/C"
 			(at 31.496 102.108 90)
 			(show_name no)
