File: BMS/ECAD/PackController/CAN.kicad_sch (KiCad schematic)
At the start: 12 parts, among them U2 MCP2562-E-SN, U3 MCP2562-E-SN

Commit message: finished schemativ of precharge
Other:
- company: (none) -> Lukas Elektronik
- title: (none) -> PackController
Changed lines of the file:
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@@
 	(generator_version "10.0")
 	(paper "A4")
+	(title_block
+		(title "PackController")
+		(date "2026-03-03")
+		(rev "V0.9")
+		(company "Lukas Elektronik")
+	)
 	(rectangle
 		(start 167.64 60.96)
