File: BMS/ECAD/PackController/CAN.kicad_sch (KiCad schematic)
At the start: 12 parts, among them U2 MCP2562-E-SN, U3 MCP2562-E-SN

Commit message: schematic finished, review tbd
Parts:
- removed C2, C4: 100nF 0603 6.3V, Capacitor_SMD:C_0603_1608Metric_Pad1.08x0.95mm_HandSolder, symbol Device:C
- removed R4: 20R 0603, Resistor_SMD:R_0603_1608Metric_Pad0.98x0.95mm_HandSolder, symbol Device:R
- removed R6: 1kR 0603, Resistor_SMD:R_0603_1608Metric_Pad0.98x0.95mm_HandSolder, symbol Device:R
- removed R8: 120R 0603, Resistor_SMD:R_0603_1608Metric_Pad0.98x0.95mm_HandSolder, symbol Device:R
- removed U3: MCP2562-E-SN, Package_SO:SOIC-8_3.9x4.9mm_P1.27mm, symbol Interface_CAN_LIN:MCP2562-E-SN
Connections:
- net CAN1_N renamed CAN_N
- net CAN1_P renamed CAN_P
- net CAN1_RX renamed CAN_RX
- net CAN1_TX renamed CAN_TX

Commit message: close to finish BMS master, only some footprints needed
Parts:
- added D501, D502: DESD5V0S1BA-7, Diode_SMD:D_SOD-323, symbol Device:D_Schottky
- renumbered C1 to C501, C3 to C502, R3 to R501, R7 to R502, R5 to R503, U2 to U501
Connections:
- net CAN_N: now also D502.1 (K)
- net CAN_P: now also D501.1 (K)
- net GND: now also D501.2 (A), D502.2 (A)

Commit message: finalised schematic of pack controller
Parts:
- C501, C502: value 100nF 0603 6.3V -> 100nF 0603 16V
Changed lines of the file:
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@@
 			)
 		)
-		(property "Value" "100nF 0603 6.3V"
+		(property "Value" "100nF 0603 16V"
 			(at 114.3 69.85 90)
 			(show_name no)
@@
 			)
 		)
-		(property "Value" "100nF 0603 6.3V"
+		(property "Value" "100nF 0603 16V"
 			(at 132.08 69.85 90)
 			(show_name no)

Commit message: yes
Parts:
- D501, D502: symbol Device:D_Schottky -> Device:D_TVS
Changed lines of the file:
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@@
 	)
 	(symbol
-		(lib_id "Device:D_Schottky")
+		(lib_id "Device:D_TVS")
 		(at 181.61 67.31 0)
 		(unit 1)
@@
 			)
 		)
-		(property "Description" ""
+		(property "Description" "Bidirectional transient-voltage-suppression diode"
 			(at 181.61 67.31 0)
+			(hide yes)
 			(show_name no)
 			(do_not_autoplace no)
@@
 	)
 	(symbol
-		(lib_id "Device:D_Schottky")
+		(lib_id "Device:D_TVS")
 		(at 181.61 63.5 0)
 		(unit 1)
@@
 			)
 		)
-		(property "Description" ""
+		(property "Description" "Bidirectional transient-voltage-suppression diode"
 			(at 181.61 63.5 0)
-			(show_name no)
-			(do_not_autoplace no)
+			(hide yes)
+			(show_name no)
+			(do_not_autoplace no)
