File: BMS/ECAD/PackController/HV_Measurement.kicad_sch (KiCad schematic)
At the start: 0 parts

Commit message: finished schemativ of precharge
Other:
- company: (none) -> Lukas Elektronik
- title: (none) -> PackController
Changed lines of the file:
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@@
 	(generator_version "10.0")
 	(paper "A4")
+	(title_block
+		(title "PackController")
+		(date "2026-03-03")
+		(rev "V0.9")
+		(company "Lukas Elektronik")
+	)
 	(image
 		(at 447.04 116.84)
