File: BMS/ECAD/PackController/Precharge.kicad_sch (KiCad schematic)
At the start: 0 parts

Commit message: finished schemativ of precharge
Parts:
- added C22, C24, C27: 100nF 0603 100V, Capacitor_SMD:C_0603_1608Metric_Pad1.08x0.95mm_HandSolder, symbol Device:C
- added C23: 47uF 1206 25V, Capacitor_SMD:C_0603_1608Metric_Pad1.08x0.95mm_HandSolder, symbol Device:C
- added C25, C26: 10uF 0603 50V, Capacitor_SMD:C_0603_1608Metric_Pad1.08x0.95mm_HandSolder, symbol Device:C
- added D403, D404: BAS16HT1G, Diode_SMD:D_SOD-323F, symbol Device:D
- added D6, D8, D9: BY2000, Diode_THT:D_DO-201AE_P12.70mm_Horizontal, symbol Device:D
- added D7: S1MB-13-F, Diode_SMD:D_SMB, symbol Device:D
- added K1: KT12-1A-40L-THT, symbol Relay:Relay_SPST-NO
- added Q6: IRLML0100TR, Package_TO_SOT_SMD:SOT-23-3, symbol Simulation_SPICE:NMOS
- added Q7: IXTA08N100D2HV, EKartParts:TO-263HV, symbol Transistor_FET_Other:Q_NMOS_Depletion_GSD
- added Q8: BC846, Package_TO_SOT_SMD:SOT-23, symbol Transistor_BJT:BC846
- added Q9: DMP4065S-7, Package_TO_SOT_SMD:SOT-23-3, symbol Simulation_SPICE:PMOS
- added R48: 47R 0603, Resistor_SMD:R_0603_1608Metric_Pad0.98x0.95mm_HandSolder, symbol Device:R
- added R50, R51, R53: 10kR 0603, Resistor_SMD:R_0603_1608Metric_Pad0.98x0.95mm_HandSolder, symbol Device:R
- added R52: 1kR 0603, Resistor_SMD:R_0603_1608Metric_Pad0.98x0.95mm_HandSolder, symbol Device:R
- added R54: 1kR 0805, Resistor_SMD:R_0603_1608Metric_Pad0.98x0.95mm_HandSolder, symbol Device:R
- added R55, R56, R57, R58: 10kR, Resistor_SMD:R_0603_1608Metric_Pad0.98x0.95mm_HandSolder, symbol Device:R
- added TH1, TH2: PTCEL17R501TBE, Varistor:RV_Disc_D16.5mm_W6.7mm_P7.5mm, symbol Device:Thermistor_PTC
- added U7, U8: TCLT1004, Package_SO:SOP-4_7.5x4.1mm_P2.54mm, symbol Isolator:Optocoupler_DC_PhotoNPN_AKEC
- added U9: TEA1-0505HI, Converter_DCDC:Converter_DCDC_TRACO_TEA1-xxxxHI_THT, symbol Converter_DCDC:TEA1-0505HI
Connections:
- new net: D9.1 (K), TH1.1
- new net: D8.1 (K), D9.2 (A)
- new net: C25.2, U9.2 (-Vin)
- new net: TH1.2, TH2.1
- new net: Q9.2 (G), R55.2, R56.1
- new net: Q8.3 (C), R56.2
- new net: C22.1, C24.1, K1.14, Q6.3 (S), Q7.1 (G), R48.2, R51.2, U8.2
- new net: Q6.1 (D), Q7.2 (S), R48.1
- new net: Q7.3 (D), TH2.2
- new net: C23.1, D403.1 (K), D404.1 (K), K1.A1
- new net: R54.1, U7.2
- new net: D7.1 (K), R52.1, U7.4
- new net: R52.2, U8.1
- new net: Q8.1 (B), R57.1
- new net: C26.2, C27.1, U9.5 (-Vout)
- new net: D6.1 (K), D7.2 (A)
- new net: C22.2, C24.2, Q6.2 (G), R50.1
- new net: R50.2, R51.1, U7.3
- new net +3.3V: U8.4
- new net +5V: C25.1, U9.1 (+Vin)
- new net +5V_TS_P_VEHI: C26.1, C27.2, D6.2 (A), U9.7 (+Vout)
- new net AIR_P_Power: Q9.1 (D)
- new net AIR_P_Switch: R57.2, R58.1
- new net GND: C23.2, D404.2 (A), K1.A2, Q8.2 (E), R53.2, R54.2, R58.2
- new net PCHRG_ACT: R53.1, U8.3
- new net SC_END: D403.2 (A), Q9.3 (S), R55.1, U7.1
- new net TS_P_ACCU: D8.2 (A)
- new net TS_P_VEHI: K1.13
Other:
- company: (none) -> Lukas Elektronik
- title: (none) -> PackController
