File: BMS/ECAD/PackController/Precharge.kicad_sch (KiCad schematic)
At the start: 38 parts, among them K1101 KT12-1A-40L-THT, Q1101 DMP4065S-7, Q1102 IXTA08N100D2HV, Q1103 BC846, Q1104 IRLML0100TR, U1101 TCLT1004, U1102 TCLT1004, U1103 TEA1-0505HI, U1104 SN74LVC2G14DBV

Commit message: yes
Parts:
- removed Q1101: DMP4065S-7, Package_TO_SOT_SMD:SOT-23-3, symbol Transistor_FET:Q_PMOS_GSD
- added Q1105: FDN352AP, Package_TO_SOT_SMD:SOT-23, symbol Lukas:FDN352AP
- C1103: value 10uF 0805 25V -> 10uF 0805 35V
- C1106: value 10uF 0805 50V -> 10uF 0805 35V
Connections:
- net PCHRG_Enable: now also Q1105.3 (D)
- net SC_END: now also Q1105.2 (S)
- net at R1101.2, R1102.1: now also Q1105.1 (G)
Changed lines of the file:
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@@
 			(justify right bottom)
 		)
-		(property "Netzklasse" "LOCAL_P_VEHI"
+		(property "Netclass" "LOCAL_P_VEHI"
 			(at 52.7685 50.8 0)
 			(show_name no)
@@
 			(justify right bottom)
 		)
-		(property "Netzklasse" "P_VEHI_+5"
+		(property "Netclass" "P_VEHI_+5"
 			(at 32.4485 154.94 0)
 			(show_name no)
@@
 			(justify right bottom)
 		)
-		(property "Netzklasse" "HV800"
+		(property "Netclass" "HV800"
 			(at 34.9885 15.24 0)
 			(show_name no)
@@
 			)
 		)
-		(property "Value" "10uF 0805 50V"
+		(property "Value" "10uF 0805 35V"
 			(at 103.886 192.786 90)
 			(show_name no)
@@
 	)
 	(symbol
-		(lib_id "Transistor_FET:Q_PMOS_GSD")
-		(at 163.83 34.29 0)
-		(mirror x)
-		(unit 1)
-		(body_style 1)
-		(exclude_from_sim no)
-		(in_bom yes)
-		(on_board yes)
-		(in_pos_files yes)
-		(dnp no)
-		(property "Reference" "Q1101"
-			(at 170.18 35.5601 0)
-			(show_name no)
-			(do_not_autoplace no)
-			(effects
-				(font
-					(size 1.27 1.27)
-				)
-				(justify left)
-			)
-		)
-		(property "Value" "DMP4065S-7"
-			(at 170.18 33.0201 0)
-			(show_name no)
-			(do_not_autoplace no)
-			(effects
-				(font
-					(size 1.27 1.27)
-				)
-				(justify left)
-			)
-		)
-		(property "Footprint" "Package_TO_SOT_SMD:SOT-23-3"
-			(at 168.91 36.83 0)
-			(hide yes)
-			(show_name no)
-			(do_not_autoplace no)
-			(effects
-				(font
-					(size 1.27 1.27)
-				)
-			)
-		)
-		(property "Datasheet" ""
-			(at 163.83 34.29 0)
-			(hide yes)
-			(show_name no)
-			(do_not_autoplace no)
-			(effects
-				(font
-					(size 1.27 1.27)
-				)
-			)
-		)
-		(property "Description" "P-MOSFET transistor, gate/source/drain"
-			(at 163.83 34.29 0)
-			(hide yes)
-			(show_name no)
-			(do_not_autoplace no)
-			(effects
-				(font
-					(size 1.27 1.27)
-				)
-			)
-		)
-		(pin "3"
-		)
-		(pin "1"
-		)
-		(pin "2"
-		)
-		(instances
-			(project "Pack_Controller"
-				(path "/58a1c93e-baba-4d23-9191-955e00968735/10db8ab2-a069-4c18-98c6-f1c7e2899a80"
-					(reference "Q1101")
-					(unit 1)
-				)
-			)
-		)
-	)
-	(symbol
 		(lib_id "Device:R")
 		(at 138.43 55.88 0)
@@
 			)
 		)
-		(property "Value" "10uF 0805 25V"
+		(property "Value" "10uF 0805 35V"
 			(at 105.664 159.766 90)
 			(show_name no)
@@
 					(unit 1)
 				)
+			)
+		)
+	)
+	(symbol
+		(lib_id "Lukas:FDN352AP")
+		(at 158.75 34.29 0)
+		(mirror x)
+		(unit 1)
+		(body_style 1)
+		(exclude_from_sim no)
+		(in_bom yes)
+		(on_board yes)
+		(in_pos_files yes)
+		(dnp no)
+		(property "Reference" "Q1105"
+			(at 170.18 34.925 0)
+			(show_name no)
+			(do_not_autoplace no)
+			(effects
+				(font
+					(size 1.524 1.524)
+				)
+				(justify left)
+			)
+		)
+		(property "Value" "FDN352AP"
+			(at 170.18 32.385 0)
+			(show_name no)
+			(do_not_autoplace no)
+			(effects
+				(font
+					(size 1.524 1.524)
+				)
+				(justify left)
+			)
+		)
+		(property "Footprint" "Package_TO_SOT_SMD:SOT-23"
+			(at 158.75 34.29 0)
+			(hide yes)
+			(show_name no)
+			(do_not_autoplace no)
+			(effects
+				(font
+					(size 1.27 1.27)
+					(italic yes)
+				)
+			)
+		)
+		(property "Datasheet" "https://www.onsemi.com/download/data-sheet/pdf/fdn352ap-d.pdf"
+			(at 158.75 34.29 0)
+			(hide yes)
+			(show_name no)
+			(do_not_autoplace no)
+			(effects
+				(font
+					(size 1.27 1.27)
+					(italic yes)
+				)
+			)
+		)
+		(property "Description" ""
+			(at 158.75 34.29 0)
+			(show_name no)
+			(do_not_autoplace no)
+			(effects
+				(font
+					(size 1.27 1.27)
+				)
+			)
+		)
+		(pin "1"
+		)
+		(pin "2"
+		)
+		(pin "3"
+		)
+		(instances
+			(project "Pack_Controller"
+				(path "/58a1c93e-baba-4d23-9191-955e00968735/10db8ab2-a069-4c18-98c6-f1c7e2899a80"
+					(reference "Q1105")
+					(unit 1)
+				)
