File: BMS/ECAD/PackController/StackCommInterface.kicad_sch (KiCad schematic)
At the start: 0 parts

Commit message: pack controller close to finished and startet pack controller
Parts:
- added C10, C11, C12, C17: 220pC 1000V, Capacitor_SMD:C_1206_3216Metric, symbol Device:C
- added C13: 330nF 16V, Capacitor_SMD:C_1206_3216Metric, symbol Device:C
- added C14, C15, C16: 100nF 16V, Capacitor_SMD:C_1206_3216Metric, symbol Device:C
- added C6, C64, C65, C66, C67, C7, C8, C9: 2.2nC 1000V, Capacitor_SMD:C_1206_3216Metric, symbol Device:C
- added R18, R19, R28, R29: 39R, Resistor_SMD:R_0603_1608Metric, symbol Device:R
- added R20, R21, R22, R23, R26, R27: 1kR, Resistor_SMD:R_0603_1608Metric, symbol Device:R
- added R24: 1.5kR, Resistor_SMD:R_0603_1608Metric, symbol Device:R
- added R25: 5.1R, Resistor_SMD:R_0603_1608Metric, symbol Device:R
- added T1, T2: HM2116ANL, symbol Device:Transformer_1P_1S
- added U1: (no value), symbol EKartParts:TLE9015
Connections:
- new net: C14.1, C15.1, U1.30 (VIO), U1.31 (VregOut_VDDA)
- new net: C17.1, C9.1, R29.1
- new net: C16.1, R25.1, U1.34 (VS), U1.35 (VS)
- new net: C65.1, C7.2
- new net: C65.2, R20.1, T1.3 (SA)
- new net: C64.2, R20.2, T1.4 (SB)
- new net: C6.2, C64.1
- new net: C10.1, C6.1, R18.1
- new net: R18.2, U1.25 (IFH_H)
- new net: R29.2, U1.23 (IFL_L)
- new net: R28.2, U1.24 (IFL_H)
- new net: R19.2, U1.26 (IFH_L)
- new net: C11.1, C8.1, R28.1
- new net: C67.2, R27.1, T2.3 (SA)
- new net: C66.2, R27.2, T2.4 (SB)
- new net: C12.1, C7.1, R19.1
- new net: C67.1, C9.2
- new net: C66.1, C8.2
- new net +BATT: R25.2
- new net ERRQ: U1.33 (ERRQ)
- new net ERRQ_Ioc_out: U1.21 (ERRQ_Ioc_out)
- new net ERRQ_ext: U1.18 (ERRQ_ext)
- new net ERRQ_ext_out: R24.2, U1.20 (ERRQ_ext_out)
- new net ERRQ_res: U1.16 (ERRQ_res)
- new net GND: C10.2, C11.2, C12.2, C13.2, C14.2, C15.2, C16.2, C17.2, U1.22 (GND), U1.49 (EP)
- new net IFH_H: R21.2, T1.1 (AA)
- new net IFH_L: R21.1, T1.2 (AB)
- new net IFL_H: R26.2, T2.1 (AA)
- new net IFL_L: R26.1, T2.2 (AB)
- new net UART_HS_RX: R23.2, U1.29 (UART_HS)
- new net UART_HS_TX: R23.1
- new net UART_LS_RX: R22.2, U1.28 (UART_LS)
- new net UART_LS_TX: R22.1
- new net VDDC: C13.1, R24.1, U1.27 (VDDC)
- new net nSleep: U1.14 (nSleep)

Commit message: finished schemativ of precharge
Other:
- title: (none) -> PackController
Changed lines of the file:
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@@
 	(paper "A4")
 	(title_block
+		(title "PackController")
 		(date "2026-03-03")
 		(rev "V0.9")
