File: BMS/ECAD/PackController/TSAL_Logik.kicad_sch (KiCad schematic)
At the start: 0 parts

Commit message: finished schemativ of precharge
Parts:
- added Q14: FDN352AP, SOT23_527AG_ONS, symbol Lukas:FDN352AP
- added Q5: BC846, Package_TO_SOT_SMD:SOT-23, symbol Transistor_BJT:BC846
- added R45, R46, R47: 10kR 0603, Resistor_SMD:R_0603_1608Metric_Pad0.98x0.95mm_HandSolder, symbol Device:R
Connections:
- new net: Q5.1 (B), R47.1
- new net: Q5.3 (C), R45.1, R46.1
- new net: Q14.1 (G), R45.2
- new net +BATT: Q14.2 (S), R46.2
- new net GND: Q5.2 (E)
- new net TSAL_GRN: Q14.3 (D)
- new net TSAL_GRN_ON: R47.2
Other:
- company: (none) -> Lukas Elektronik
- title: (none) -> PackController
