File: BMS/ECAD/PackController/Supply.kicad_sch (KiCad schematic)
At the start: 12 parts, among them U15 R-78E3.3-1.0, U16 R-78E5.0-1.0

Commit message: close to finish BMS master, only some footprints needed
Parts:
- renumbered 3V3Good1 to 3V3Good1801, 5VGood1 to 5VGood1801, C43 to C1801, C44 to C1802, C45 to C1803, C46 to C1804, C47 to C1805, C48 to C1806, R55 to R1801, R56 to R1802, U15 to U1801, U16 to U1802
Changed lines of the file:
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@@
 		(dnp no)
 		(fields_autoplaced yes)
-		(property "Reference" "3V3Good1"
+		(property "Reference" "3V3Good1801"
 			(at 104.14 116.5225 90)
 			(show_name no)
@@
 			(project "Pack_Controller"
 				(path "/58a1c93e-baba-4d23-9191-955e00968735/967a6172-dcc3-4702-8f77-1a76e5d988cf"
-					(reference "3V3Good1")
+					(reference "3V3Good1801")
 					(unit 1)
 				)
@@
 		(dnp no)
 		(fields_autoplaced yes)
-		(property "Reference" "#PWR058"
+		(property "Reference" "#PWR01804"
 			(at 231.14 102.87 0)
 			(hide yes)
@@
 			(project "Pack_Controller"
 				(path "/58a1c93e-baba-4d23-9191-955e00968735/967a6172-dcc3-4702-8f77-1a76e5d988cf"
-					(reference "#PWR058")
+					(reference "#PWR01804")
 					(unit 1)
 				)
@@
 		(in_pos_files yes)
 		(dnp no)
-		(property "Reference" "C47"
+		(property "Reference" "C1805"
 			(at 180.34 106.68 0)
 			(show_name no)
@@
 			(project "Pack_Controller"
 				(path "/58a1c93e-baba-4d23-9191-955e00968735/967a6172-dcc3-4702-8f77-1a76e5d988cf"
-					(reference "C47")
+					(reference "C1805")
 					(unit 1)
 				)
@@
 		(in_pos_files yes)
 		(dnp no)
-		(property "Reference" "#PWR057"
+		(property "Reference" "#PWR01807"
 			(at 201.93 129.54 0)
 			(hide yes)
@@
 			(project "Pack_Controller"
 				(path "/58a1c93e-baba-4d23-9191-955e00968735/967a6172-dcc3-4702-8f77-1a76e5d988cf"
-					(reference "#PWR057")
+					(reference "#PWR01807")
 					(unit 1)
 				)
@@
 		(dnp no)
 		(fields_autoplaced yes)
-		(property "Reference" "5VGood1"
+		(property "Reference" "5VGood1801"
 			(at 234.95 117.7925 90)
 			(show_name no)
@@
 			(project "Pack_Controller"
 				(path "/58a1c93e-baba-4d23-9191-955e00968735/967a6172-dcc3-4702-8f77-1a76e5d988cf"
-					(reference "5VGood1")
+					(reference "5VGood1801")
 					(unit 1)
 				)
@@
 		(in_pos_files yes)
 		(dnp no)
-		(property "Reference" "#PWR039"
+		(property "Reference" "#PWR01806"
 			(at 69.85 128.27 0)
 			(hide yes)
@@
 			(project "Pack_Controller"
 				(path "/58a1c93e-baba-4d23-9191-955e00968735/967a6172-dcc3-4702-8f77-1a76e5d988cf"
-					(reference "#PWR039")
+					(reference "#PWR01806")
 					(unit 1)
 				)
@@
 		(in_pos_files yes)
 		(dnp no)
-		(property "Reference" "C46"
+		(property "Reference" "C1804"
 			(at 120.65 109.22 0)
 			(show_name no)
@@
 			(project "Pack_Controller"
 				(path "/58a1c93e-baba-4d23-9191-955e00968735/967a6172-dcc3-4702-8f77-1a76e5d988cf"
-					(reference "C46")
+					(reference "C1804")
 					(unit 1)
 				)
@@
 		(dnp no)
 		(fields_autoplaced yes)
-		(property "Reference" "U15"
+		(property "Reference" "U1801"
 			(at 69.85 95.25 0)
 			(show_name no)
@@
 			(project "Pack_Controller"
 				(path "/58a1c93e-baba-4d23-9191-955e00968735/967a6172-dcc3-4702-8f77-1a76e5d988cf"
-					(reference "U15")
+					(reference "U1801")
 					(unit 1)
 				)
@@
 		(in_pos_files yes)
 		(dnp no)
-		(property "Reference" "C44"
+		(property "Reference" "C1802"
 			(at 58.42 113.03 0)
 			(show_name no)
@@
 			(project "Pack_Controller"
 				(path "/58a1c93e-baba-4d23-9191-955e00968735/967a6172-dcc3-4702-8f77-1a76e5d988cf"
-					(reference "C44")
+					(reference "C1802")
 					(unit 1)
 				)
@@
 		(in_pos_files yes)
 		(dnp no)
-		(property "Reference" "#PWR054"
+		(property "Reference" "#PWR01805"
 			(at 118.11 121.92 0)
 			(hide yes)
@@
 			(project "Pack_Controller"
 				(path "/58a1c93e-baba-4d23-9191-955e00968735/967a6172-dcc3-4702-8f77-1a76e5d988cf"
-					(reference "#PWR054")
+					(reference "#PWR01805")
 					(unit 1)
 				)
@@
 		(in_pos_files yes)
 		(dnp no)
-		(property "Reference" "R55"
+		(property "Reference" "R1801"
 			(at 107.95 105.41 0)
 			(show_name no)
@@
 			(project "Pack_Controller"
 				(path "/58a1c93e-baba-4d23-9191-955e00968735/967a6172-dcc3-4702-8f77-1a76e5d988cf"
-					(reference "R55")
+					(reference "R1801")
 					(unit 1)
 				)
@@
 		(dnp no)
 		(fields_autoplaced yes)
-		(property "Reference" "#PWR055"
+		(property "Reference" "#PWR01802"
 			(at 116.84 101.6 0)
 			(hide yes)
@@
 			(project "Pack_Controller"
 				(path "/58a1c93e-baba-4d23-9191-955e00968735/967a6172-dcc3-4702-8f77-1a76e5d988cf"
-					(reference "#PWR055")
+					(reference "#PWR01802")
 					(unit 1)
 				)
@@
 		(in_pos_files yes)
 		(dnp no)
-		(property "Reference" "C48"
+		(property "Reference" "C1806"
 			(at 223.52 106.68 0)
 			(show_name no)
@@
 			(project "Pack_Controller"
 				(path "/58a1c93e-baba-4d23-9191-955e00968735/967a6172-dcc3-4702-8f77-1a76e5d988cf"
-					(reference "C48")
+					(reference "C1806")
 					(unit 1)
 				)
@@
 		(dnp no)
 		(fields_autoplaced yes)
-		(property "Reference" "#PWR056"
+		(property "Reference" "#PWR01803"
 			(at 194.31 102.87 0)
 			(hide yes)
@@
 			(project "Pack_Controller"
 				(path "/58a1c93e-baba-4d23-9191-955e00968735/967a6172-dcc3-4702-8f77-1a76e5d988cf"
-					(reference "#PWR056")
+					(reference "#PWR01803")
 					(unit 1)
 				)
@@
 		(dnp no)
 		(fields_autoplaced yes)
-		(property "Reference" "#PWR034"
+		(property "Reference" "#PWR01801"
 			(at 55.88 101.6 0)
 			(hide yes)
@@
 			(project "Pack_Controller"
 				(path "/58a1c93e-baba-4d23-9191-955e00968735/967a6172-dcc3-4702-8f77-1a76e5d988cf"
-					(reference "#PWR034")
+					(reference "#PWR01801")
 					(unit 1)
 				)
@@
 		(in_pos_files yes)
 		(dnp no)
-		(property "Reference" "C43"
+		(property "Reference" "C1801"
 			(at 46.99 106.68 0)
 			(show_name no)
@@
 			(project "Pack_Controller"
 				(path "/58a1c93e-baba-4d23-9191-955e00968735/967a6172-dcc3-4702-8f77-1a76e5d988cf"
-					(reference "C43")
+					(reference "C1801")
 					(unit 1)
 				)
@@
 		(in_pos_files yes)
 		(dnp no)
-		(property "Reference" "C45"
+		(property "Reference" "C1803"
 			(at 91.44 105.41 0)
 			(show_name no)
@@
 			(project "Pack_Controller"
 				(path "/58a1c93e-baba-4d23-9191-955e00968735/967a6172-dcc3-4702-8f77-1a76e5d988cf"
-					(reference "C45")
+					(reference "C1803")
 					(unit 1)
 				)
@@
 		(in_pos_files yes)
 		(dnp no)
-		(property "Reference" "R56"
+		(property "Reference" "R1802"
 			(at 238.76 106.68 0)
 			(show_name no)
@@
 			(project "Pack_Controller"
 				(path "/58a1c93e-baba-4d23-9191-955e00968735/967a6172-dcc3-4702-8f77-1a76e5d988cf"
-					(reference "R56")
+					(reference "R1802")
 					(unit 1)
 				)
@@
 		(dnp no)
 		(fields_autoplaced yes)
-		(property "Reference" "U16"
+		(property "Reference" "U1802"
 			(at 201.93 96.52 0)
 			(show_name no)
@@
 			(project "Pack_Controller"
 				(path "/58a1c93e-baba-4d23-9191-955e00968735/967a6172-dcc3-4702-8f77-1a76e5d988cf"
-					(reference "U16")
-					(unit 1)
-				)
+					(reference "U1802")
+					(unit 1)
+				)

Commit message: finalised schematic of pack controller
Parts:
- C1801: value 470uF 16V WE870025374007 -> 470uF 35V WE870025374007
- C1802, C1803, C1805, C1806: value 10uF 0805 16V -> 10uF 0805 35V
- C1804: value 100uF 16V WE870025374007 -> 100uF 35V WE870025374007
Changed lines of the file:
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@@
 		)
 	)
-	(text_box "+5V Supply worst-case estimate:\n\nMain loads:\nTEA1-0505HI isolated DC/DC no-load, 3x:    ~84 mA\nTEA1 loads incl. ADuM3190 isolated sides:  ~25...30 mA\nMCP2562 CAN transceivers, 2x dominant:     ~140 mA\nMisc. reserve / startup / tolerance:       ~50 mA\n\nEstimated worst-case load:                 ~250...300 mA\nSelected supply: RECOM 5 V / 1 A DC/DC\n\nDesign margin:\n1 A / 300 mA ≈ 3.3x"
+	(text_box "+5V Supply worst-case estimate:\n\nMain loads:\nTEA1-0505HI isolated DC/DC no-load, 5x:    ~120 mA\nTEA1 loads incl. ADuM3190 isolated sides:  ~25...30 mA\nMCP2562 CAN transceivers, 2x dominant:     ~140 mA\nMisc. reserve / startup / tolerance:       ~50 mA\n\nEstimated worst-case load:                 ~330...400 mA\nSelected supply: RECOM 5 V / 1 A DC/DC\n\nDesign margin:\nDesign margin: 1A / 0.4A ≈ 2.5x"
 		(exclude_from_sim no)
 		(at 186.69 69.85 0)
@@
 			)
 		)
-		(property "Value" "10uF 0805 16V"
+		(property "Value" "10uF 0805 35V"
 			(at 175.26 109.22 0)
 			(show_name no)
@@
 			)
 		)
-		(property "Value" "100uF 16V WE870025374007"
+		(property "Value" "100uF 35V WE870025374007"
 			(at 119.38 111.76 0)
 			(show_name no)
@@
 			)
 		)
-		(property "Value" "10uF 0805 16V"
+		(property "Value" "10uF 0805 35V"
 			(at 53.34 115.57 0)
 			(show_name no)
@@
 			)
 		)
-		(property "Value" "10uF 0805 16V"
+		(property "Value" "10uF 0805 35V"
 			(at 228.6 109.22 0)
 			(show_name no)
@@
 			)
 		)
-		(property "Value" "470uF 16V WE870025374007"
+		(property "Value" "470uF 35V WE870025374007"
 			(at 22.86 109.22 0)
 			(show_name no)
@@
 			)
 		)
-		(property "Value" "10uF 0805 16V"
+		(property "Value" "10uF 0805 35V"
 			(at 96.52 107.95 0)
 			(show_name no)
