File: BMS/ECAD/PackController/MCU.kicad_sch (KiCad schematic)
At the start: 54 parts, among them Q201 DMP4065S-7, Q202 BC846, U201 MCP130-270, U203 SN74LVC1G74, U204 STM32G483VET6, U205 24LC256-I/SN, Y201 WE830055951

Commit message: finalised schematic of pack controller
Parts:
- U201: value MCP130-270 -> MCP130-270 ITT
- U202: value (none) -> STWD100YNYWY; footprint (none) -> Package_TO_SOT_SMD:SOT-23-5
- Y201: footprint Oscillator:Oscillator_SMD_EuroQuartz_XO32-4Pin_3.2x2.5mm_HandSoldering -> Oscillator:Oscillator_SMD_EuroQuartz_XO32-4Pin_3.2x2.5mm
Other:
- moved on the sheet: C213, U203B
Changed lines of the file:
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@@
 	(text_box "SC latch / reset / watchdog logic:\n\nU201 MCP130 generates nPOR from +3.3V.\nnPOR is used only as power-on/brownout set signal for U203A.\n\nPower-up / brownout:\nnPOR = LOW\n-> U203A nPRE = LOW\n-> Q = HIGH\n-> Q202/Q201 enable SC_Out\n-> D201 also pulls nRES LOW and keeps MCU in reset\n\nAfter nPOR release:\nnPOR = HIGH\n-> U203A keeps previous Q state\n-> MCU starts via nRES release\n\nU202 watchdog:\nnWDO = LOW on watchdog fault\n-> D203 pulls nRES LOW\n-> D207 pulls U203A nCLR LOW\n-> Q = LOW\n-> SC_Out disabled / opened\n\nLatch_SC:\nMCU can pull Latch_SC LOW\n-> D206 pulls U203A nCLR LOW\n-> Q = LOW\n-> SC_Out disabled / opened\n\nImportant:\nnPOR, nRES and nWDO are diode-isolated.\nnRES must not pull nPOR or nCLR LOW.\nThis avoids simultaneous nPRE/nCLR activation of U203A.\n\nRe-closing SC after watchdog fault or Latch_SC clear requires power-cycle / nPOR event.\nSC_State is derived from U203A Q and indicates actual latch output state."
 		(exclude_from_sim no)
-		(at 269.24 33.02 0)
-		(size 74.93 63.0817)
+		(at 231.14 99.1383 0)
+		(size 52.07 64.6917)
 		(margins 0.9525 0.9525 0.9525 0.9525)
 		(stroke
@@
 	)
 	(junction
-		(at 260.35 138.43)
+		(at 165.1 189.23)
 		(diameter 0)
 		(color 0 0 0 0)
@@
 	)
 	(junction
-		(at 241.3 134.62)
+		(at 146.05 185.42)
 		(diameter 0)
 		(color 0 0 0 0)
@@
 	(wire
 		(pts
-			(xy 241.3 134.62) (xy 242.57 134.62)
+			(xy 146.05 185.42) (xy 147.32 185.42)
 		)
 		(stroke
@@
 	(wire
 		(pts
-			(xy 260.35 138.43) (xy 260.35 134.62)
+			(xy 165.1 189.23) (xy 165.1 185.42)
 		)
 		(stroke
@@
 	(wire
 		(pts
-			(xy 254 143.51) (xy 260.35 143.51)
+			(xy 158.75 194.31) (xy 165.1 194.31)
 		)
 		(stroke
@@
 	(wire
 		(pts
-			(xy 246.38 143.51) (xy 241.3 143.51)
+			(xy 151.13 194.31) (xy 146.05 194.31)
 		)
 		(stroke
@@
 	(wire
 		(pts
-			(xy 260.35 143.51) (xy 260.35 138.43)
+			(xy 165.1 194.31) (xy 165.1 189.23)
 		)
 		(stroke
@@
 	(wire
 		(pts
-			(xy 260.35 134.62) (xy 259.08 134.62)
+			(xy 165.1 185.42) (xy 163.83 185.42)
 		)
 		(stroke
@@
 	(wire
 		(pts
-			(xy 241.3 133.35) (xy 241.3 134.62)
+			(xy 146.05 184.15) (xy 146.05 185.42)
 		)
 		(stroke
@@
 	(wire
 		(pts
-			(xy 241.3 143.51) (xy 241.3 134.62)
+			(xy 146.05 194.31) (xy 146.05 185.42)
 		)
 		(stroke
@@
 		(in_pos_files yes)
 		(dnp no)
-		(fields_autoplaced yes)
 		(property "Reference" "U202"
 			(at 197.231 41.91 0)
@@
 			)
 		)
-		(property "Value" ""
-			(at 189.23 27.94 0)
+		(property "Value" "STWD100YNYWY"
+			(at 182.372 28.702 0)
 			(show_name no)
 			(do_not_autoplace no)
@@
 			)
 		)
-		(property "Footprint" ""
+		(property "Footprint" "Package_TO_SOT_SMD:SOT-23-5"
 			(at 189.23 27.94 0)
 			(hide yes)
@@
 			)
 		)
-		(property "Datasheet" ""
+		(property "Datasheet" "https://www.st.com/resource/en/datasheet/stwd100.pdf"
 			(at 189.23 27.94 0)
 			(hide yes)
@@
 	(symbol
 		(lib_id "power:GND")
-		(at 260.35 138.43 90)
+		(at 165.1 189.23 90)
 		(unit 1)
 		(body_style 1)
@@
 		(dnp no)
 		(property "Reference" "#PWR0223"
-			(at 266.7 138.43 0)
+			(at 171.45 189.23 0)
 			(hide yes)
 			(show_name no)
@@
 		)
 		(property "Value" "GND"
-			(at 264.16 138.43 0)
+			(at 168.91 189.23 0)
 			(show_name no)
 			(do_not_autoplace no)
@@
 		)
 		(property "Footprint" ""
-			(at 260.35 138.43 0)
+			(at 165.1 189.23 0)
 			(hide yes)
 			(show_name no)
@@
 		)
 		(property "Datasheet" ""
-			(at 260.35 138.43 0)
+			(at 165.1 189.23 0)
 			(hide yes)
 			(show_name no)
@@
 		)
 		(property "Description" ""
-			(at 260.35 138.43 0)
+			(at 165.1 189.23 0)
 			(show_name no)
 			(do_not_autoplace no)
@@
 	(symbol
 		(lib_id "EKartParts:SN74LVC1G74")
-		(at 251.46 118.11 0)
+		(at 156.21 168.91 0)
 		(unit 2)
 		(body_style 1)
@@
 		(dnp no)
 		(property "Reference" "U203"
-			(at 250.825 130.81 0)
+			(at 155.575 181.61 0)
 			(show_name no)
 			(do_not_autoplace no)
@@
 		)
 		(property "Value" "SN74LVC1G74"
-			(at 250.952 137.16 0)
+			(at 155.702 187.96 0)
 			(show_name no)
 			(do_not_autoplace no)
@@
 		)
 		(property "Footprint" "Package_SO:VSSOP-8_2.3x2mm_P0.5mm"
-			(at 251.46 118.11 0)
+			(at 156.21 168.91 0)
 			(hide yes)
 			(show_name no)
@@
 		)
 		(property "Datasheet" ""
-			(at 251.46 118.11 0)
+			(at 156.21 168.91 0)
 			(hide yes)
 			(show_name no)
@@
 		)
 		(property "Description" ""
-			(at 251.46 118.11 0)
+			(at 156.21 168.91 0)
 			(hide yes)
 			(show_name no)
@@
 			)
 		)
-		(property "Value" "MCP130-270"
+		(property "Value" "MCP130-270 ITT"
 			(at 148.59 36.83 90)
 			(show_name no)
@@
 	(symbol
 		(lib_id "Device:C")
-		(at 250.19 143.51 270)
+		(at 154.94 194.31 270)
 		(unit 1)
 		(body_style 1)
@@
 		(dnp no)
 		(property "Reference" "C213"
-			(at 248.412 139.954 90)
+			(at 153.162 190.754 90)
 			(show_name no)
 			(do_not_autoplace no)
@@
 		)
 		(property "Value" "100nF 0603 6.3V"
-			(at 251.46 145.034 90)
+			(at 156.21 195.834 90)
 			(show_name no)
 			(do_not_autoplace no)
@@
 		)
 		(property "Footprint" "Capacitor_SMD:C_0603_1608Metric_Pad1.08x0.95mm_HandSolder"
-			(at 246.38 144.4752 0)
+			(at 151.13 195.2752 0)
 			(hide yes)
 			(show_name no)
@@
 		)
 		(property "Datasheet" ""
-			(at 250.19 143.51 0)
+			(at 154.94 194.31 0)
 			(hide yes)
 			(show_name no)
@@
 		)
 		(property "Description" ""
-			(at 250.19 143.51 0)
+			(at 154.94 194.31 0)
 			(show_name no)
 			(do_not_autoplace no)
@@
 			)
 		)
-		(property "Footprint" "Oscillator:Oscillator_SMD_EuroQuartz_XO32-4Pin_3.2x2.5mm_HandSoldering"
+		(property "Footprint" "Oscillator:Oscillator_SMD_EuroQuartz_XO32-4Pin_3.2x2.5mm"
 			(at 25.4 62.23 0)
 			(hide yes)
@@
 	(symbol
 		(lib_id "power:+3.3V")
-		(at 241.3 133.35 0)
+		(at 146.05 184.15 0)
 		(unit 1)
 		(body_style 1)
@@
 		(dnp no)
 		(property "Reference" "#PWR0222"
-			(at 241.3 137.16 0)
+			(at 146.05 187.96 0)
 			(hide yes)
 			(show_name no)
@@
 		)
 		(property "Value" "+3.3V"
-			(at 241.3 129.54 0)
+			(at 146.05 180.34 0)
 			(show_name no)
 			(do_not_autoplace no)
@@
 		)
 		(property "Footprint" ""
-			(at 241.3 133.35 0)
+			(at 146.05 184.15 0)
 			(hide yes)
 			(show_name no)
@@
 		)
 		(property "Datasheet" ""
-			(at 241.3 133.35 0)
+			(at 146.05 184.15 0)
 			(hide yes)
 			(show_name no)
@@
 		)
 		(property "Description" ""
-			(at 241.3 133.35 0)
+			(at 146.05 184.15 0)
 			(show_name no)
 			(do_not_autoplace no)

Commit message: many fixes
Parts:
- removed JP201, JP202: Jumper_2_Open, Jumper:SolderJumper-2_P1.3mm_Open_RoundedPad1.0x1.5mm, symbol Jumper:Jumper_2_Open
Connections:
- net +3.3V: now also U204.36 (VREF+)
- net AIR_Error renamed nAIR_Error
Changed lines of the file:
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@@
 	)
 	(junction
-		(at 77.47 50.8)
-		(diameter 0)
-		(color 0 0 0 0)
-	)
-	(junction
 		(at 107.95 43.18)
 		(diameter 0)
@@
 	(wire
 		(pts
-			(xy 55.88 41.91) (xy 64.77 41.91)
-		)
-		(stroke
-			(width 0)
-			(type default)
-		)
-	)
-	(wire
-		(pts
 			(xy 158.75 194.31) (xy 165.1 194.31)
 		)
@@
 	(wire
 		(pts
-			(xy 74.93 41.91) (xy 77.47 41.91)
-		)
-		(stroke
-			(width 0)
-			(type default)
-		)
-	)
-	(wire
-		(pts
 			(xy 154.94 53.34) (xy 125.73 53.34)
 		)
@@
 	(wire
 		(pts
-			(xy 77.47 50.8) (xy 82.55 50.8)
-		)
-		(stroke
-			(width 0)
-			(type default)
-		)
-	)
-	(wire
-		(pts
 			(xy 154.94 149.86) (xy 125.73 149.86)
 		)
@@
 	(wire
 		(pts
-			(xy 77.47 41.91) (xy 77.47 50.8)
-		)
-		(stroke
-			(width 0)
-			(type default)
-		)
-	)
-	(wire
-		(pts
 			(xy 156.21 124.46) (xy 142.24 124.46)
 		)
@@
 	(wire
 		(pts
-			(xy 74.93 50.8) (xy 77.47 50.8)
-		)
-		(stroke
-			(width 0)
-			(type default)
-		)
-	)
-	(wire
-		(pts
 			(xy 31.75 80.01) (xy 31.75 87.63)
 		)
@@
 	(wire
 		(pts
-			(xy 64.77 50.8) (xy 63.5 50.8)
+			(xy 80.01 50.8) (xy 82.55 50.8)
 		)
 		(stroke
@@
 		)
 	)
-	(label "VREF+"
-		(at 55.88 41.91 0)
-		(effects
-			(font
-				(size 1.27 1.27)
-			)
-			(justify left bottom)
-		)
-	)
 	(label "WP1"
 		(at 224.79 138.43 180)
@@
 		)
 	)
-	(hierarchical_label "AIR_Error"
+	(hierarchical_label "nAIR_Error"
 		(shape input)
 		(at 154.94 111.76 0)
@@
 	)
 	(symbol
-		(lib_id "Jumper:Jumper_2_Open")
-		(at 69.85 41.91 180)
-		(unit 1)
-		(body_style 1)
-		(exclude_from_sim no)
-		(in_bom yes)
-		(on_board yes)
-		(in_pos_files yes)
-		(dnp no)
-		(property "Reference" "JP201"
-			(at 67.31 36.83 0)
-			(show_name no)
-			(do_not_autoplace no)
-			(effects
-				(font
-					(size 1.27 1.27)
-				)
-				(justify right)
-			)
-		)
-		(property "Value" "Jumper_2_Open"
-			(at 62.23 39.37 0)
-			(show_name no)
-			(do_not_autoplace no)
-			(effects
-				(font
-					(size 1.27 1.27)
-				)
-				(justify right)
-			)
-		)
-		(property "Footprint" "Jumper:SolderJumper-2_P1.3mm_Open_RoundedPad1.0x1.5mm"
-			(at 69.85 41.91 0)
-			(hide yes)
-			(show_name no)
-			(do_not_autoplace no)
-			(effects
-				(font
-					(size 1.27 1.27)
-				)
-			)
-		)
-		(property "Datasheet" ""
-			(at 69.85 41.91 0)
-			(hide yes)
-			(show_name no)
-			(do_not_autoplace no)
-			(effects
-				(font
-					(size 1.27 1.27)
-				)
-			)
-		)
-		(property "Description" ""
-			(at 69.85 41.91 0)
-			(show_name no)
-			(do_not_autoplace no)
-			(effects
-				(font
-					(size 1.27 1.27)
-				)
-			)
-		)
-		(pin "1"
-		)
-		(pin "2"
-		)
-		(instances
-			(project "Pack_Controller"
-				(path "/58a1c93e-baba-4d23-9191-955e00968735/e566c49f-462b-40b2-a95e-665611e574ab"
-					(reference "JP201")
-					(unit 1)
-				)
-			)
-		)
-	)
-	(symbol
 		(lib_id "power:+3.3V")
 		(at 210.82 86.36 0)
@@
 	)
 	(symbol
-		(lib_id "Jumper:Jumper_2_Open")
-		(at 69.85 50.8 180)
-		(unit 1)
-		(body_style 1)
-		(exclude_from_sim no)
-		(in_bom yes)
-		(on_board yes)
-		(in_pos_files yes)
-		(dnp no)
-		(property "Reference" "JP202"
-			(at 67.31 45.72 0)
-			(show_name no)
-			(do_not_autoplace no)
-			(effects
-				(font
-					(size 1.27 1.27)
-				)
-				(justify right)
-			)
-		)
-		(property "Value" "Jumper_2_Open"
-			(at 62.23 48.26 0)
-			(show_name no)
-			(do_not_autoplace no)
-			(effects
-				(font
-					(size 1.27 1.27)
-				)
-				(justify right)
-			)
-		)
-		(property "Footprint" "Jumper:SolderJumper-2_P1.3mm_Open_RoundedPad1.0x1.5mm"
-			(at 69.85 50.8 0)
-			(hide yes)
-			(show_name no)
-			(do_not_autoplace no)
-			(effects
-				(font
-					(size 1.27 1.27)
-				)
-			)
-		)
-		(property "Datasheet" ""
-			(at 69.85 50.8 0)
-			(hide yes)
-			(show_name no)
-			(do_not_autoplace no)
-			(effects
-				(font
-					(size 1.27 1.27)
-				)
-			)
-		)
-		(property "Description" ""
-			(at 69.85 50.8 0)
-			(show_name no)
-			(do_not_autoplace no)
-			(effects
-				(font
-					(size 1.27 1.27)
-				)
-			)
-		)
-		(pin "1"
-		)
-		(pin "2"
-		)
-		(instances
-			(project "Pack_Controller"
-				(path "/58a1c93e-baba-4d23-9191-955e00968735/e566c49f-462b-40b2-a95e-665611e574ab"
-					(reference "JP202")
-					(unit 1)
-				)
-			)
-		)
-	)
-	(symbol
 		(lib_id "power:GND")
 		(at 173.99 114.3 0)
@@
 	(symbol
 		(lib_id "power:+3.3V")
-		(at 63.5 50.8 90)
+		(at 80.01 50.8 90)
 		(unit 1)
 		(body_style 1)
@@
 		(dnp no)
 		(property "Reference" "#PWR0212"
-			(at 67.31 50.8 0)
+			(at 83.82 50.8 0)
 			(hide yes)
 			(show_name no)
@@
 		)
 		(property "Value" "+3.3V"
-			(at 57.15 50.8 90)
+			(at 73.66 50.8 90)
 			(show_name no)
 			(do_not_autoplace no)
@@
 		)
 		(property "Footprint" ""
-			(at 63.5 50.8 0)
+			(at 80.01 50.8 0)
 			(hide yes)
 			(show_name no)
@@
 		)
 		(property "Datasheet" ""
-			(at 63.5 50.8 0)
+			(at 80.01 50.8 0)
 			(hide yes)
 			(show_name no)
@@
 		)
 		(property "Description" ""
-			(at 63.5 50.8 0)
+			(at 80.01 50.8 0)
 			(show_name no)
 			(do_not_autoplace no)

Commit message: add rule areas for hv separation
Parts:
- C208: value 100nF 0603 6.3V -> 100nF 0603 16V
Changed lines of the file:
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@@
 			)
 		)
-		(property "Value" "100nF 0603 6.3V"
+		(property "Value" "100nF 0603 16V"
 			(at 197.866 25.4 90)
 			(show_name no)
