File: BMS/ECAD/PackController/AIR.kicad_sch (KiCad schematic)
At the start: 33 parts, among them K401 AIR_N, K402 AIR_P, Q401 DMP4065S-7, Q402 BC846, Q403 DMP4065S-7, Q404 BC846, U401 ADCMP393ARZ

Commit message: many fixes
Connections:
- net AIR_N_AUX1: now also U401.11 (+); no longer U401.10 (-)
- net AIR_P_AUX1: now also U401.7 (+); no longer U401.6 (-)
- net at R408.1, R410.2: now also U401.10 (-), U401.6 (-); no longer U401.11 (+), U401.7 (+)
- net AIR_Error renamed nAIR_Error
- net DANGER_V renamed DANGER_V_oD
Changed lines of the file:
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@@
 	)
 	(junction
+		(at 45.72 165.1)
+		(diameter 0)
+		(color 0 0 0 0)
+	)
+	(junction
 		(at 54.61 80.01)
 		(diameter 0)
@@
 	)
 	(junction
-		(at 49.53 165.1)
+		(at 64.77 36.83)
 		(diameter 0)
 		(color 0 0 0 0)
 	)
 	(junction
-		(at 64.77 36.83)
+		(at 49.53 165.1)
 		(diameter 0)
 		(color 0 0 0 0)
@@
 	)
 	(junction
-		(at 45.72 165.1)
-		(diameter 0)
-		(color 0 0 0 0)
-	)
-	(junction
 		(at 38.1 49.53)
 		(diameter 0)
@@
 	)
 	(junction
-		(at 146.05 63.5)
+		(at 121.92 107.95)
 		(diameter 0)
 		(color 0 0 0 0)
 	)
 	(junction
-		(at 121.92 107.95)
+		(at 187.96 60.96)
 		(diameter 0)
 		(color 0 0 0 0)
 	)
 	(junction
-		(at 187.96 60.96)
+		(at 33.02 176.53)
 		(diameter 0)
 		(color 0 0 0 0)
 	)
 	(junction
-		(at 33.02 176.53)
+		(at 146.05 63.5)
 		(diameter 0)
 		(color 0 0 0 0)
@@
 	(wire
 		(pts
-			(xy 59.69 170.18) (xy 59.69 176.53)
-		)
-		(stroke
-			(width 0)
-			(type default)
-		)
-	)
-	(wire
-		(pts
-			(xy 146.05 29.21) (xy 146.05 30.48)
+			(xy 127 58.42) (xy 146.05 58.42)
 		)
 		(stroke
@@
 	(wire
 		(pts
-			(xy 182.88 124.46) (xy 182.88 130.81)
+			(xy 59.69 170.18) (xy 59.69 176.53)
 		)
 		(stroke
@@
 	(wire
 		(pts
-			(xy 64.77 36.83) (xy 78.74 36.83)
+			(xy 146.05 29.21) (xy 146.05 30.48)
 		)
 		(stroke
@@
 	(wire
 		(pts
-			(xy 146.05 58.42) (xy 168.91 58.42)
+			(xy 182.88 124.46) (xy 182.88 130.81)
 		)
 		(stroke
@@
 	(wire
 		(pts
-			(xy 146.05 58.42) (xy 146.05 63.5)
+			(xy 64.77 36.83) (xy 78.74 36.83)
 		)
 		(stroke
@@
 	(wire
 		(pts
-			(xy 45.72 161.29) (xy 45.72 165.1)
+			(xy 45.72 151.13) (xy 45.72 165.1)
 		)
 		(stroke
@@
 	(wire
 		(pts
+			(xy 139.7 63.5) (xy 127 63.5)
+		)
+		(stroke
+			(width 0)
+			(type default)
+		)
+	)
+	(wire
+		(pts
 			(xy 182.88 104.14) (xy 184.15 104.14)
 		)
@@
 	(wire
 		(pts
-			(xy 107.95 33.02) (xy 107.95 34.29)
+			(xy 146.05 63.5) (xy 168.91 63.5)
 		)
 		(stroke
@@
 	(wire
 		(pts
-			(xy 59.69 158.75) (xy 59.69 160.02)
+			(xy 107.95 33.02) (xy 107.95 34.29)
 		)
 		(stroke
@@
 	(wire
 		(pts
-			(xy 43.18 22.86) (xy 43.18 21.59)
+			(xy 59.69 158.75) (xy 59.69 160.02)
 		)
 		(stroke
@@
 	(wire
 		(pts
-			(xy 49.53 161.29) (xy 49.53 165.1)
+			(xy 43.18 22.86) (xy 43.18 21.59)
 		)
 		(stroke
@@
 	(wire
 		(pts
-			(xy 156.21 63.5) (xy 168.91 63.5)
-		)
-		(stroke
-			(width 0)
-			(type default)
-		)
-	)
-	(wire
-		(pts
 			(xy 46.99 21.59) (xy 50.8 21.59)
 		)
@@
 	(wire
 		(pts
-			(xy 139.7 58.42) (xy 127 58.42)
-		)
-		(stroke
-			(width 0)
-			(type default)
-		)
-	)
-	(wire
-		(pts
 			(xy 101.6 107.95) (xy 101.6 119.38)
 		)
@@
 	(wire
 		(pts
-			(xy 127 63.5) (xy 146.05 63.5)
+			(xy 259.08 66.04) (xy 274.32 66.04)
 		)
 		(stroke
@@
 	(wire
 		(pts
-			(xy 259.08 66.04) (xy 274.32 66.04)
+			(xy 50.8 53.34) (xy 50.8 54.61)
 		)
 		(stroke
@@
 	(wire
 		(pts
-			(xy 50.8 53.34) (xy 50.8 54.61)
+			(xy 38.1 46.99) (xy 38.1 49.53)
 		)
 		(stroke
@@
 	(wire
 		(pts
-			(xy 38.1 46.99) (xy 38.1 49.53)
+			(xy 43.18 165.1) (xy 45.72 165.1)
 		)
 		(stroke
@@
 	(wire
 		(pts
-			(xy 43.18 165.1) (xy 45.72 165.1)
+			(xy 156.21 58.42) (xy 168.91 58.42)
 		)
 		(stroke
@@
 	(wire
 		(pts
+			(xy 146.05 63.5) (xy 146.05 66.04)
+		)
+		(stroke
+			(width 0)
+			(type default)
+		)
+	)
+	(wire
+		(pts
 			(xy 121.92 107.95) (xy 119.38 107.95)
 		)
@@
 	(wire
 		(pts
-			(xy 146.05 63.5) (xy 146.05 66.04)
+			(xy 146.05 58.42) (xy 146.05 63.5)
 		)
 		(stroke
@@
 		)
 	)
+	(wire
+		(pts
+			(xy 49.53 151.13) (xy 49.53 165.1)
+		)
+		(stroke
+			(width 0)
+			(type default)
+		)
+	)
 	(label "AIR_P_Enable"
 		(at 78.74 39.37 180)
@@
 		)
 	)
-	(label "AIR_N_AUX1"
-		(at 139.7 58.42 180)
-		(effects
-			(font
-				(size 1.27 1.27)
-			)
-			(justify right bottom)
-		)
-	)
 	(label "AIR_P_AUX1"
 		(at 156.21 45.72 0)
@@
 		)
 	)
-	(label "AIR_P_AUX1"
-		(at 156.21 63.5 0)
+	(label "AIR_N_AUX1"
+		(at 231.14 41.91 0)
 		(effects
 			(font
@@
 	)
 	(label "AIR_N_AUX1"
-		(at 231.14 41.91 0)
+		(at 139.7 63.5 180)
 		(effects
 			(font
 				(size 1.27 1.27)
 			)
-			(justify left bottom)
+			(justify right bottom)
 		)
 	)
@@
 		)
 	)
+	(label "AIR_P_AUX1"
+		(at 156.21 58.42 0)
+		(effects
+			(font
+				(size 1.27 1.27)
+			)
+			(justify left bottom)
+		)
+	)
 	(label "AIR_P_Enable"
 		(at 82.55 157.48 180)
@@
 		)
 	)
-	(hierarchical_label "DANGER_V"
+	(hierarchical_label "DANGER_V_oD"
 		(shape input)
-		(at 49.53 161.29 90)
+		(at 49.53 151.13 90)
 		(effects
 			(font
@@
 		)
 	)
-	(hierarchical_label "AIR_Error"
+	(hierarchical_label "nAIR_Error"
 		(shape input)
 		(at 110.49 60.96 180)
@@
 		)
 	)
-	(hierarchical_label "AIR_Error"
+	(hierarchical_label "nAIR_Error"
 		(shape input)
 		(at 189.23 60.96 0)
@@
 	(hierarchical_label "PRCHG_DONE"
 		(shape input)
-		(at 45.72 161.29 90)
+		(at 45.72 151.13 90)
 		(effects
 			(font
@@
 		(in_pos_files yes)
 		(dnp no)
-		(fields_autoplaced yes)
 		(property "Reference" "#PWR0404"
 			(at 107.95 36.83 0)
@@
 		)
 		(property "Value" "+3.3V"
-			(at 107.95 27.94 0)
+			(at 107.95 29.21 0)
 			(show_name no)
 			(do_not_autoplace no)
@@
 			)
 		)
-		(property "Datasheet" ""
+		(property "Datasheet" "https://www.analog.com/media/en/technical-documentation/data-sheets/ADCMP391_392_393.pdf"
 			(at 171.45 38.1 0)
 			(hide yes)
@@
 			)
 		)
-		(property "Datasheet" ""
+		(property "Datasheet" "https://www.analog.com/media/en/technical-documentation/data-sheets/ADCMP391_392_393.pdf"
 			(at 124.46 66.04 0)
 			(hide yes)
@@
 			)
 		)
-		(property "Datasheet" ""
+		(property "Datasheet" "https://www.analog.com/media/en/technical-documentation/data-sheets/ADCMP391_392_393.pdf"
 			(at 124.46 48.26 0)
 			(hide yes)
@@
 		(in_pos_files yes)
 		(dnp no)
-		(fields_autoplaced yes)
 		(property "Reference" "#PWR0405"
 			(at 187.96 36.83 0)
@@
 		)
 		(property "Value" "+3.3V"
-			(at 187.96 27.94 0)
+			(at 187.96 29.21 0)
 			(show_name no)
 			(do_not_autoplace no)
@@
 		(in_pos_files yes)
 		(dnp no)
-		(fields_autoplaced yes)
 		(property "Reference" "#PWR0401"
 			(at 46.99 24.13 0)
@@
 		)
 		(property "Value" "+3.3V"
-			(at 46.99 15.24 0)
+			(at 46.736 16.764 0)
 			(show_name no)
 			(do_not_autoplace no)
@@
 		(in_pos_files yes)
 		(dnp no)
-		(fields_autoplaced yes)
 		(property "Reference" "#PWR0407"
 			(at 38.1 62.23 0)
@@
 		)
 		(property "Value" "GND"
-			(at 38.1 60.96 0)
+			(at 38.1 59.69 0)
 			(show_name no)
 			(do_not_autoplace no)
@@
 		(in_pos_files yes)
 		(dnp no)
-		(fields_autoplaced yes)
 		(property "Reference" "#PWR0403"
 			(at 146.05 33.02 0)
@@
 		)
 		(property "Value" "+3.3V"
-			(at 146.05 24.13 0)
+			(at 146.05 25.146 0)
 			(show_name no)
 			(do_not_autoplace no)
@@
 			)
 		)
-		(property "Datasheet" ""
+		(property "Datasheet" "https://www.analog.com/media/en/technical-documentation/data-sheets/ADCMP391_392_393.pdf"
 			(at 116.84 111.76 0)
 			(hide yes)
@@
 			)
 		)
-		(property "Datasheet" ""
+		(property "Datasheet" "https://www.analog.com/media/en/technical-documentation/data-sheets/ADCMP391_392_393.pdf"
 			(at 171.45 55.88 0)
 			(hide yes)

Commit message: add rule areas for hv separation
Changed lines of the file:
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@@
+	)
+	(junction
+		(at 54.61 80.01)
+		(diameter 0)
+		(color 0 0 0 0)
+	)
+	(junction
+		(at 163.83 130.81)
+		(diameter 0)
+		(color 0 0 0 0)
+	)
+	(junction
+		(at 146.05 40.64)
+		(diameter 0)
+		(color 0 0 0 0)
+	)
+	(junction
+		(at 59.69 139.7)
+		(diameter 0)
+		(color 0 0 0 0)
+	)
+	(junction
+		(at 46.99 21.59)
+		(diameter 0)
+		(color 0 0 0 0)
+	)
+	(junction
+		(at 64.77 36.83)
+		(diameter 0)
+		(color 0 0 0 0)
+	)
+	(junction
+		(at 58.42 54.61)
+		(diameter 0)
+		(color 0 0 0 0)
+	)
+	(junction
+		(at 59.69 149.86)
+		(diameter 0)
+		(color 0 0 0 0)
+	)
+	(junction
+		(at 33.02 165.1)
+		(diameter 0)
+		(color 0 0 0 0)
+	)
+	(junction
+		(at 182.88 93.98)
+		(diameter 0)
+		(color 0 0 0 0)
+	)
+	(junction
+		(at 38.1 54.61)
+		(diameter 0)
+		(color 0 0 0 0)
+	)
+	(junction
+		(at 58.42 39.37)
+		(diameter 0)
+		(color 0 0 0 0)
+	)
+	(junction
+		(at 107.95 43.18)
+		(diameter 0)
+		(color 0 0 0 0)
+	)
+	(junction
+		(at 146.05 45.72)
+		(diameter 0)
+		(color 0 0 0 0)
+	)
+	(junction
+		(at 38.1 49.53)
+		(diameter 0)
+		(color 0 0 0 0)
+	)
+	(junction
+		(at 163.83 119.38)
+		(diameter 0)
+		(color 0 0 0 0)
+	)
+	(junction
+		(at 50.8 54.61)
+		(diameter 0)
+		(color 0 0 0 0)
+	)
+	(junction
+		(at 49.53 165.1)
+		(diameter 0)
+		(color 0 0 0 0)
+	)
+	(junction
+		(at 121.92 107.95)
+		(diameter 0)
+		(color 0 0 0 0)
 	)
 	(junction
@@
 	)
 	(junction
-		(at 54.61 80.01)
-		(diameter 0)
-		(color 0 0 0 0)
-	)
-	(junction
-		(at 163.83 130.81)
-		(diameter 0)
-		(color 0 0 0 0)
-	)
-	(junction
-		(at 146.05 40.64)
-		(diameter 0)
-		(color 0 0 0 0)
-	)
-	(junction
-		(at 59.69 139.7)
-		(diameter 0)
-		(color 0 0 0 0)
-	)
-	(junction
-		(at 46.99 21.59)
-		(diameter 0)
-		(color 0 0 0 0)
-	)
-	(junction
-		(at 64.77 36.83)
-		(diameter 0)
-		(color 0 0 0 0)
-	)
-	(junction
-		(at 49.53 165.1)
-		(diameter 0)
-		(color 0 0 0 0)
-	)
-	(junction
-		(at 58.42 54.61)
-		(diameter 0)
-		(color 0 0 0 0)
-	)
-	(junction
-		(at 59.69 149.86)
-		(diameter 0)
-		(color 0 0 0 0)
-	)
-	(junction
-		(at 33.02 165.1)
-		(diameter 0)
-		(color 0 0 0 0)
-	)
-	(junction
-		(at 182.88 93.98)
-		(diameter 0)
-		(color 0 0 0 0)
-	)
-	(junction
-		(at 38.1 54.61)
-		(diameter 0)
-		(color 0 0 0 0)
-	)
-	(junction
-		(at 58.42 39.37)
-		(diameter 0)
-		(color 0 0 0 0)
-	)
-	(junction
-		(at 107.95 43.18)
-		(diameter 0)
-		(color 0 0 0 0)
-	)
-	(junction
-		(at 146.05 45.72)
-		(diameter 0)
-		(color 0 0 0 0)
-	)
-	(junction
-		(at 38.1 49.53)
-		(diameter 0)
-		(color 0 0 0 0)
-	)
-	(junction
-		(at 163.83 119.38)
-		(diameter 0)
-		(color 0 0 0 0)
-	)
-	(junction
-		(at 50.8 54.61)
-		(diameter 0)
-		(color 0 0 0 0)
-	)
-	(junction
-		(at 121.92 107.95)
-		(diameter 0)
-		(color 0 0 0 0)
-	)
-	(junction
 		(at 187.96 60.96)
 		(diameter 0)
@@
 	(wire
 		(pts
-			(xy 45.72 151.13) (xy 45.72 165.1)
+			(xy 45.72 162.56) (xy 45.72 165.1)
 		)
 		(stroke
@@
 	(wire
 		(pts
-			(xy 49.53 151.13) (xy 49.53 165.1)
+			(xy 49.53 162.56) (xy 49.53 165.1)
 		)
 		(stroke
@@
 	(hierarchical_label "DANGER_V_oD"
 		(shape input)
-		(at 49.53 151.13 90)
+		(at 49.53 162.56 90)
 		(effects
 			(font
@@
 	(hierarchical_label "PRCHG_DONE"
 		(shape input)
-		(at 45.72 151.13 90)
-		(effects
-			(font
+		(at 45.72 162.56 90)
+		(effects
+			(font

Commit message: yes
Changed lines of the file:
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@@
 	(rectangle
 		(start 213.36 12.7)
-		(end 284.48 85.09)
+		(end 284.48 86.36)
 		(stroke
 			(width 0)
