File: BMS/ECAD/PackController/Buzzer.kicad_sch (KiCad schematic)
At the start: 5 parts, among them Q15 2N7002

Commit message: schematic finished, review tbd
Parts:
- R38: value 1kR 0603 -> 10kR 0603
Changed lines of the file:
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@@
 			)
 		)
-		(property "Value" "1kR 0603"
+		(property "Value" "10kR 0603"
 			(at 136.144 106.68 0)
 			(show_name no)

Commit message: close to finish BMS master, only some footprints needed
Parts:
- renumbered Q15 to Q801, R36 to R801, R37 to R802, R35 to R803, R38 to R804
Changed lines of the file:
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@@
 		(in_pos_files yes)
 		(dnp no)
-		(property "Reference" "R38"
+		(property "Reference" "R804"
 			(at 129.54 106.68 90)
 			(show_name no)
@@
 			(project "Pack_Controller"
 				(path "/58a1c93e-baba-4d23-9191-955e00968735/9e76a46f-aff0-416c-bf65-690935f0ea58"
-					(reference "R38")
+					(reference "R804")
 					(unit 1)
 				)
@@
 		(in_pos_files yes)
 		(dnp no)
-		(property "Reference" "Q15"
+		(property "Reference" "Q801"
 			(at 148.59 100.965 0)
 			(show_name no)
@@
 			(project "Pack_Controller"
 				(path "/58a1c93e-baba-4d23-9191-955e00968735/9e76a46f-aff0-416c-bf65-690935f0ea58"
-					(reference "Q15")
+					(reference "Q801")
 					(unit 1)
 				)
@@
 		(in_pos_files yes)
 		(dnp no)
-		(property "Reference" "R37"
+		(property "Reference" "R802"
 			(at 144.78 78.74 90)
 			(show_name no)
@@
 			(project "Pack_Controller"
 				(path "/58a1c93e-baba-4d23-9191-955e00968735/9e76a46f-aff0-416c-bf65-690935f0ea58"
-					(reference "R37")
+					(reference "R802")
 					(unit 1)
 				)
@@
 		(in_pos_files yes)
 		(dnp no)
-		(property "Reference" "R36"
+		(property "Reference" "R801"
 			(at 138.176 72.39 90)
 			(show_name no)
@@
 			(project "Pack_Controller"
 				(path "/58a1c93e-baba-4d23-9191-955e00968735/9e76a46f-aff0-416c-bf65-690935f0ea58"
-					(reference "R36")
+					(reference "R801")
 					(unit 1)
 				)
@@
 		(in_pos_files yes)
 		(dnp no)
-		(property "Reference" "R35"
+		(property "Reference" "R803"
 			(at 121.92 100.33 90)
 			(show_name no)
@@
 			(project "Pack_Controller"
 				(path "/58a1c93e-baba-4d23-9191-955e00968735/9e76a46f-aff0-416c-bf65-690935f0ea58"
-					(reference "R35")
+					(reference "R803")
 					(unit 1)
 				)
@@
 		(in_pos_files yes)
 		(dnp no)
-		(property "Reference" "#PWR016"
+		(property "Reference" "#PWR0802"
 			(at 144.78 119.38 0)
 			(hide yes)
@@
 			(project "Pack_Controller"
 				(path "/58a1c93e-baba-4d23-9191-955e00968735/9e76a46f-aff0-416c-bf65-690935f0ea58"
-					(reference "#PWR016")
+					(reference "#PWR0802")
 					(unit 1)
 				)
@@
 		(dnp no)
 		(fields_autoplaced yes)
-		(property "Reference" "#PWR038"
+		(property "Reference" "#PWR0801"
 			(at 130.81 72.39 0)
 			(hide yes)
@@
 			(project "Pack_Controller"
 				(path "/58a1c93e-baba-4d23-9191-955e00968735/9e76a46f-aff0-416c-bf65-690935f0ea58"
-					(reference "#PWR038")
-					(unit 1)
-				)
+					(reference "#PWR0801")
+					(unit 1)
+				)

Commit message: many fixes
Changed lines of the file:
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@@
 		(dnp no)
 		(property "Reference" "R801"
-			(at 138.176 72.39 90)
+			(at 138.43 72.39 90)
 			(show_name no)
 			(do_not_autoplace no)

Commit message: yes
Changed lines of the file:
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@@
 		(company "Lukas Elektronik")
 	)
-	(text_box "Passive piezo buzzer driver.\nTarget part: CPT-2305-90PM, externally driven, 12 Vp-p, 4 kHz, typ. 24 nF.\n\nDrive with STM32 PWM:\nf_PWM ≈ 4 kHz\nduty ≈ 50 %\n\nQ15 is a low-side NMOS switch.\nR37 discharges the piezo during MOSFET off-time:\ntau = R37 * C_PIEZO ≈ 2.2k * 24nF ≈ 53us.\n\nR36 limits peak current and EMI.\nNo additional series coupling capacitor required."
+	(text_box "Passive piezo buzzer driver.\nTarget: CPT-2305-90PM, 12 Vp-p, 4 kHz, C_PIEZO typ. 24 nF.\n\nQ801 = low-side NMOS, driven by STM32 PWM:\nf ~= 4 kHz, duty ~= 50 %\n\nR801 = 100R limits capacitive peak current:\nI_peak <= VBATT,max / R801 = 16V / 100R = 160 mA\ntau_ON = R801 * C_PIEZO = 2.4 us\n\nR802 = 2.2k discharges piezo:\ntau_OFF = R802 * C_PIEZO = 52.8 us\nAt 4 kHz: t_OFF ~= 125 us\nV_remain ~= exp(-125us / 52.8us) = 9.4 %\n\nFET current check:\nI_Q801,rms ~= 12 mA incl. R802 discharge/load current.\nEven with RDS(on) = 100R:\nP_Q801 ~= 14 mW"
 		(exclude_from_sim no)
 		(at 167.64 78.7669 0)
-		(size 62.23 22.8331)
+		(size 62.23 32.4928)
 		(margins 0.9525 0.9525 0.9525 0.9525)
 		(stroke
