File: BMS/ECAD/PackController/DCDC_AIR.kicad_sch (KiCad schematic)
At the start: 35 parts, among them K1901 KT12-1A-40L-THT, Q1901 IXTA08N100D2HV, Q1902 IPD95R750P7, Q1903 BC846, Q1904 DMP4065S-7, U1901 TCLT1004, U1902 TCLT1004, U1903 TEA1-0505HI, U1904 SN74LVC2G14DBV

Commit message: most of layout complete
Parts:
- added D1903: BY2000, Diode_THT:D_DO-201AE_P12.70mm_Horizontal, symbol Device:D
Connections:
- net +5V_TS_P_DCDC: now also D1903.2 (A); no longer R1904.1, U1901.4
- new net: D1903.1 (K), R1904.1, U1901.4
Changed lines of the file:
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@@
 	(wire
 		(pts
-			(xy 67.31 36.83) (xy 67.31 82.55)
+			(xy 67.31 36.83) (xy 67.31 54.61)
 		)
 		(stroke
@@
 	(wire
 		(pts
+			(xy 67.31 62.23) (xy 67.31 82.55)
+		)
+		(stroke
+			(width 0)
+			(type default)
+		)
+	)
+	(wire
+		(pts
 			(xy 255.27 147.32) (xy 255.27 153.67)
 		)
@@
 		(polyline
 			(pts
-				(xy 76.2 48.26) (xy 30.48 48.26) (xy 27.94 48.26) (xy 27.94 151.13) (xy 76.835 151.13) (xy 76.2 62.23)
-				(xy 76.2 59.69) (xy 76.2 57.15)
+				(xy 36.83 78.74) (xy 36.83 87.63) (xy 29.21 87.63) (xy 29.21 69.85) (xy 13.97 69.85) (xy 13.97 151.13)
+				(xy 76.835 151.13) (xy 76.2 78.74)
 			)
 			(stroke
@@
 		(polyline
 			(pts
-				(xy 13.97 12.7) (xy 76.835 12.7) (xy 77.47 196.85) (xy 13.97 196.85)
+				(xy 12.7 12.7) (xy 76.835 12.7) (xy 77.47 196.85) (xy 12.7 197.485)
 			)
 			(stroke
@@
 		(length 2.54)
 		(shape round)
-		(at 44.45 48.26 180)
+		(at 48.26 78.74 180)
 		(effects
 			(font
@@
 		)
 		(property "Netzklasse" "LOCAL_P_DCDC"
-			(at 45.1485 50.8 0)
+			(at 48.9585 81.28 0)
 			(show_name no)
 			(do_not_autoplace no)
@@
 		)
 		(property "Component Class" ""
-			(at 21.59 -30.48 0)
+			(at 25.4 0 0)
 			(show_name no)
 			(do_not_autoplace no)
@@
 		(length 2.54)
 		(shape round)
-		(at 67.31 64.77 90)
-		(fields_autoplaced yes)
-		(effects
-			(font
-				(size 1.27 1.27)
-			)
-			(justify left bottom)
-		)
-		(property "Netzklasse" "HV800"
-			(at 64.77 64.0715 90)
-			(show_name no)
-			(do_not_autoplace no)
-			(effects
-				(font
-					(size 1.27 1.27)
-				)
-				(justify left)
-			)
-		)
-		(property "Component Class" ""
-			(at 44.45 -13.97 0)
-			(show_name no)
-			(do_not_autoplace no)
-			(effects
-				(font
-					(size 1.27 1.27)
-					(italic yes)
-				)
-			)
-		)
-	)
-	(netclass_flag ""
-		(length 2.54)
-		(shape round)
 		(at 17.78 12.7 180)
 		(fields_autoplaced yes)
@@
 					(unit 1)
 				)
+			)
+		)
+	)
+	(symbol
+		(lib_id "Device:D")
+		(at 67.31 58.42 90)
+		(unit 1)
+		(body_style 1)
+		(exclude_from_sim no)
+		(in_bom yes)
+		(on_board yes)
+		(in_pos_files yes)
+		(dnp no)
+		(fields_autoplaced yes)
+		(property "Reference" "D1903"
+			(at 69.85 57.1499 90)
+			(show_name no)
+			(do_not_autoplace no)
+			(effects
+				(font
+					(size 1.27 1.27)
+				)
+				(justify right)
+			)
+		)
+		(property "Value" "BY2000"
+			(at 69.85 59.6899 90)
+			(show_name no)
+			(do_not_autoplace no)
+			(effects
+				(font
+					(size 1.27 1.27)
+				)
+				(justify right)
+			)
+		)
+		(property "Footprint" "Diode_THT:D_DO-201AE_P12.70mm_Horizontal"
+			(at 67.31 58.42 0)
+			(hide yes)
+			(show_name no)
+			(do_not_autoplace no)
+			(effects
+				(font
+					(size 1.27 1.27)
+				)
+			)
+		)
+		(property "Datasheet" ""
+			(at 67.31 58.42 0)
+			(hide yes)
+			(show_name no)
+			(do_not_autoplace no)
+			(effects
+				(font
+					(size 1.27 1.27)
+				)
+			)
+		)
+		(property "Description" "Diode"
+			(at 67.31 58.42 0)
+			(hide yes)
+			(show_name no)
+			(do_not_autoplace no)
+			(effects
+				(font
+					(size 1.27 1.27)
+				)
+			)
+		)
+		(property "Sim.Device" "D"
+			(at 67.31 58.42 0)
+			(hide yes)
+			(show_name no)
+			(do_not_autoplace no)
+			(effects
+				(font
+					(size 1.27 1.27)
+				)
+			)
+		)
+		(property "Sim.Pins" "1=K 2=A"
+			(at 67.31 58.42 0)
+			(hide yes)
+			(show_name no)
+			(do_not_autoplace no)
+			(effects
+				(font
+					(size 1.27 1.27)
+				)
+			)
+		)
+		(pin "2"
+		)
+		(pin "1"
+		)
+		(instances
+			(project "Pack_Controller"
+				(path "/58a1c93e-baba-4d23-9191-955e00968735/b3a91e7b-f813-4b7e-8a66-9207449a05f0"
+					(reference "D1903")
+					(unit 1)
+				)

Commit message: yes
Parts:
- removed Q1904: DMP4065S-7, Package_TO_SOT_SMD:SOT-23-3, symbol Transistor_FET:Q_PMOS_GSD
- added Q1905: FDN352AP, Package_TO_SOT_SMD:SOT-23, symbol Lukas:FDN352AP
- C1904, C1905: value 10uF 0805 50V -> 10uF 0805 35V
- C1906: value 10uF 0805 25V -> 10uF 0805 35V
Connections:
- net DCDC_AIR_Enable: now also Q1905.3 (D)
- net SC_END: now also Q1905.2 (S)
- net at R1911.2, R1912.1: now also Q1905.1 (G)
Changed lines of the file:
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@@
 			(justify right bottom)
 		)
-		(property "Netzklasse" "LOCAL_P_DCDC"
+		(property "Netclass" "LOCAL_P_DCDC"
 			(at 48.9585 81.28 0)
 			(show_name no)
@@
 			(justify right bottom)
 		)
-		(property "Netzklasse" "P_DCDC_+5"
+		(property "Netclass" "P_DCDC_+5"
 			(at 31.1785 154.94 0)
 			(show_name no)
@@
 			(justify right bottom)
 		)
-		(property "Netzklasse" "HV800"
+		(property "Netclass" "HV800"
 			(at 18.4785 15.24 0)
 			(show_name no)
@@
 	)
 	(symbol
+		(lib_id "Lukas:FDN352AP")
+		(at 256.54 127 0)
+		(mirror x)
+		(unit 1)
+		(body_style 1)
+		(exclude_from_sim no)
+		(in_bom yes)
+		(on_board yes)
+		(in_pos_files yes)
+		(dnp no)
+		(property "Reference" "Q1905"
+			(at 267.97 127.635 0)
+			(show_name no)
+			(do_not_autoplace no)
+			(effects
+				(font
+					(size 1.524 1.524)
+				)
+				(justify left)
+			)
+		)
+		(property "Value" "FDN352AP"
+			(at 267.97 125.095 0)
+			(show_name no)
+			(do_not_autoplace no)
+			(effects
+				(font
+					(size 1.524 1.524)
+				)
+				(justify left)
+			)
+		)
+		(property "Footprint" "Package_TO_SOT_SMD:SOT-23"
+			(at 256.54 127 0)
+			(hide yes)
+			(show_name no)
+			(do_not_autoplace no)
+			(effects
+				(font
+					(size 1.27 1.27)
+					(italic yes)
+				)
+			)
+		)
+		(property "Datasheet" "https://www.onsemi.com/download/data-sheet/pdf/fdn352ap-d.pdf"
+			(at 256.54 127 0)
+			(hide yes)
+			(show_name no)
+			(do_not_autoplace no)
+			(effects
+				(font
+					(size 1.27 1.27)
+					(italic yes)
+				)
+			)
+		)
+		(property "Description" ""
+			(at 256.54 127 0)
+			(show_name no)
+			(do_not_autoplace no)
+			(effects
+				(font
+					(size 1.27 1.27)
+				)
+			)
+		)
+		(pin "1"
+		)
+		(pin "2"
+		)
+		(pin "3"
+		)
+		(instances
+			(project "Pack_Controller"
+				(path "/58a1c93e-baba-4d23-9191-955e00968735/b3a91e7b-f813-4b7e-8a66-9207449a05f0"
+					(reference "Q1905")
+					(unit 1)
+				)
+			)
+		)
+	)
+	(symbol
 		(lib_id "power:GND")
 		(at 91.44 190.5 0)
@@
 			)
 		)
-		(property "Value" "10uF 0805 50V"
+		(property "Value" "10uF 0805 35V"
 			(at 97.536 192.786 90)
 			(show_name no)
@@
 			)
 		)
-		(property "Value" "10uF 0805 25V"
+		(property "Value" "10uF 0805 35V"
 			(at 99.314 159.766 90)
 			(show_name no)
@@
 	)
 	(symbol
-		(lib_id "Transistor_FET:Q_PMOS_GSD")
-		(at 261.62 127 0)
-		(mirror x)
-		(unit 1)
-		(body_style 1)
-		(exclude_from_sim no)
-		(in_bom yes)
-		(on_board yes)
-		(in_pos_files yes)
-		(dnp no)
-		(property "Reference" "Q1904"
-			(at 267.97 128.2701 0)
-			(show_name no)
-			(do_not_autoplace no)
-			(effects
-				(font
-					(size 1.27 1.27)
-				)
-				(justify left)
-			)
-		)
-		(property "Value" "DMP4065S-7"
-			(at 267.97 125.7301 0)
-			(show_name no)
-			(do_not_autoplace no)
-			(effects
-				(font
-					(size 1.27 1.27)
-				)
-				(justify left)
-			)
-		)
-		(property "Footprint" "Package_TO_SOT_SMD:SOT-23-3"
-			(at 266.7 129.54 0)
-			(hide yes)
-			(show_name no)
-			(do_not_autoplace no)
-			(effects
-				(font
-					(size 1.27 1.27)
-				)
-			)
-		)
-		(property "Datasheet" ""
-			(at 261.62 127 0)
-			(hide yes)
-			(show_name no)
-			(do_not_autoplace no)
-			(effects
-				(font
-					(size 1.27 1.27)
-				)
-			)
-		)
-		(property "Description" "P-MOSFET transistor, gate/source/drain"
-			(at 261.62 127 0)
-			(hide yes)
-			(show_name no)
-			(do_not_autoplace no)
-			(effects
-				(font
-					(size 1.27 1.27)
-				)
-			)
-		)
-		(pin "3"
-		)
-		(pin "1"
-		)
-		(pin "2"
-		)
-		(instances
-			(project "Pack_Controller"
-				(path "/58a1c93e-baba-4d23-9191-955e00968735/b3a91e7b-f813-4b7e-8a66-9207449a05f0"
-					(reference "Q1904")
-					(unit 1)
-				)
-			)
-		)
-	)
-	(symbol
 		(lib_id "Device:R")
 		(at 242.57 142.24 270)
@@
 			)
 		)
-		(property "Value" "10uF 0805 50V"
+		(property "Value" "10uF 0805 35V"
 			(at 63.246 192.278 90)
 			(show_name no)
