File: BMS/ECAD/PackController/IMD_Monitoring.kicad_sch (KiCad schematic)
At the start: 18 parts, among them Q2301 BC846, Q2302 DMP4065S-7, Q2303 DMP4065S-7, U2301 SN74LVC1G74, U2302 SN74LVC2G14DBV

Commit message: finalised schematic of pack controller
Parts:
- removed Q2303: DMP4065S-7, Package_TO_SOT_SMD:SOT-23-3, symbol Simulation_SPICE:PMOS
- added D2303: BAT46, Diode_SMD:D_SOD-123, symbol Diode:BAT46
- C2301: footprint Capacitor_SMD:C_0603_1608Metric_Pad1.08x0.95mm_HandSolder -> Capacitor_SMD:C_0805_2012Metric
- R2305: value 1.5MR -> 39kR
- R2306: value 1.5MR -> 10kR
Connections:
- net IMD_OK: now also D2303.1 (K)
- net IMD_SC_Closed: now also D2303.2 (A)
Changed lines of the file:
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@@
 		(company "Lukas Elektronik")
 	)
+	(text_box "During IMD startup, nPRE and nCLR may overlap.\nSC_Out is forced disabled by IMD_OK low clamp.\nLatch becomes effective only after IMD_OK release."
+		(exclude_from_sim no)
+		(at 125.73 113.9163 0)
+		(size 44.45 6.7337)
+		(margins 0.9525 0.9525 0.9525 0.9525)
+		(stroke
+			(width 0)
+			(type solid)
+			(color 0 0 0 1)
+		)
+		(fill
+			(type color)
+			(color 255 255 194 1)
+		)
+		(effects
+			(font
+				(size 1 1)
+				(color 0 0 0 1)
+			)
+			(justify left top)
+		)
+	)
 	(text_box "Populate pullup/-down depending on IMD type:\nOpen-Collector: 10k Pullup + 0Ohm series resistor\nOpen-Emitter: 1k5 Pulldown + 10kOhm series resistor\n\n(Use Variants to see on schematic)"
 		(exclude_from_sim no)
@@
 	)
 	(junction
-		(at 161.29 91.44)
+		(at 134.62 106.68)
 		(diameter 0)
 		(color 0 0 0 0)
 	)
 	(junction
-		(at 245.11 44.45)
+		(at 161.29 91.44)
 		(diameter 0)
 		(color 0 0 0 0)
 	)
 	(junction
-		(at 134.62 106.68)
+		(at 245.11 44.45)
 		(diameter 0)
 		(color 0 0 0 0)
@@
 	(wire
 		(pts
+			(xy 161.29 106.68) (xy 160.02 106.68)
+		)
+		(stroke
+			(width 0)
+			(type default)
+		)
+	)
+	(wire
+		(pts
 			(xy 90.17 96.52) (xy 90.17 97.79)
 		)
@@
 	(wire
 		(pts
-			(xy 134.62 106.68) (xy 153.67 106.68)
+			(xy 134.62 106.68) (xy 152.4 106.68)
 		)
 		(stroke
@@
 	(wire
 		(pts
-			(xy 191.77 41.91) (xy 191.77 44.45)
+			(xy 161.29 91.44) (xy 161.29 106.68)
 		)
 		(stroke
@@
 	(wire
 		(pts
-			(xy 134.62 104.14) (xy 134.62 106.68)
+			(xy 191.77 41.91) (xy 191.77 44.45)
 		)
 		(stroke
@@
 	(wire
 		(pts
-			(xy 166.37 91.44) (xy 166.37 93.98)
+			(xy 134.62 104.14) (xy 134.62 106.68)
 		)
 		(stroke
@@
 	(wire
 		(pts
-			(xy 176.53 76.2) (xy 176.53 77.47)
+			(xy 166.37 91.44) (xy 166.37 93.98)
 		)
 		(stroke
@@
 	(wire
 		(pts
-			(xy 166.37 90.17) (xy 166.37 91.44)
+			(xy 176.53 76.2) (xy 176.53 77.47)
 		)
 		(stroke
@@
 	(wire
 		(pts
-			(xy 85.09 68.58) (xy 85.09 69.85)
+			(xy 166.37 90.17) (xy 166.37 91.44)
 		)
 		(stroke
@@
 	(wire
 		(pts
-			(xy 161.29 91.44) (xy 161.29 101.6)
+			(xy 85.09 68.58) (xy 85.09 69.85)
 		)
 		(stroke
@@
 	(wire
 		(pts
-			(xy 161.29 111.76) (xy 161.29 113.03)
-		)
-		(stroke
-			(width 0)
-			(type default)
-		)
-	)
-	(wire
-		(pts
 			(xy 24.13 39.37) (xy 24.13 43.18)
 		)
@@
 	)
 	(symbol
-		(lib_id "power:GND")
-		(at 161.29 113.03 0)
-		(mirror y)
-		(unit 1)
-		(body_style 1)
-		(exclude_from_sim no)
-		(in_bom yes)
-		(on_board yes)
-		(in_pos_files yes)
-		(dnp no)
-		(property "Reference" "#PWR02311"
-			(at 161.29 119.38 0)
-			(hide yes)
-			(show_name no)
-			(do_not_autoplace no)
-			(effects
-				(font
-					(size 1.27 1.27)
-				)
-			)
-		)
-		(property "Value" "GND"
-			(at 161.29 116.84 0)
-			(show_name no)
-			(do_not_autoplace no)
-			(effects
-				(font
-					(size 1.27 1.27)
-				)
-			)
-		)
-		(property "Footprint" ""
-			(at 161.29 113.03 0)
-			(hide yes)
-			(show_name no)
-			(do_not_autoplace no)
-			(effects
-				(font
-					(size 1.27 1.27)
-				)
-			)
-		)
-		(property "Datasheet" ""
-			(at 161.29 113.03 0)
-			(hide yes)
-			(show_name no)
-			(do_not_autoplace no)
-			(effects
-				(font
-					(size 1.27 1.27)
-				)
-			)
-		)
-		(property "Description" ""
-			(at 161.29 113.03 0)
-			(show_name no)
-			(do_not_autoplace no)
-			(effects
-				(font
-					(size 1.27 1.27)
-				)
-			)
-		)
-		(pin "1"
-		)
-		(instances
-			(project "Pack_Controller"
-				(path "/58a1c93e-baba-4d23-9191-955e00968735/bb6d2c27-83db-4480-8c62-fedc9a39072f"
-					(reference "#PWR02311")
-					(unit 1)
-				)
-			)
-		)
-	)
-	(symbol
 		(lib_id "EKartParts:SN74LVC1G74")
 		(at 25.4 33.02 90)
@@
 	)
 	(symbol
-		(lib_id "Simulation_SPICE:PMOS")
-		(at 158.75 106.68 0)
-		(mirror x)
-		(unit 1)
-		(body_style 1)
-		(exclude_from_sim no)
-		(in_bom yes)
-		(on_board yes)
-		(in_pos_files yes)
-		(dnp no)
-		(property "Reference" "Q2303"
-			(at 145.796 103.886 0)
-			(show_name no)
-			(do_not_autoplace no)
-			(effects
-				(font
-					(size 1.27 1.27)
-				)
-				(justify left)
-			)
-		)
-		(property "Value" "DMP4065S-7"
-			(at 145.796 101.346 0)
-			(show_name no)
-			(do_not_autoplace no)
-			(effects
-				(font
-					(size 1.27 1.27)
-				)
-				(justify left)
-			)
-		)
-		(property "Footprint" "Package_TO_SOT_SMD:SOT-23-3"
-			(at 163.83 109.22 0)
-			(hide yes)
-			(show_name no)
-			(do_not_autoplace no)
-			(effects
-				(font
-					(size 1.27 1.27)
-				)
-			)
-		)
-		(property "Datasheet" "https://ngspice.sourceforge.io/docs/ngspice-html-manual/manual.xhtml#cha_MOSFETs"
-			(at 158.75 93.98 0)
-			(hide yes)
-			(show_name no)
-			(do_not_autoplace no)
-			(effects
-				(font
-					(size 1.27 1.27)
-				)
-			)
-		)
-		(property "Description" "P-MOSFET transistor, drain/source/gate"
-			(at 158.75 106.68 0)
-			(hide yes)
-			(show_name no)
-			(do_not_autoplace no)
-			(effects
-				(font
-					(size 1.27 1.27)
-				)
-			)
-		)
-		(property "Sim.Device" "PMOS"
-			(at 158.75 89.535 0)
-			(hide yes)
-			(show_name no)
-			(do_not_autoplace no)
-			(effects
-				(font
-					(size 1.27 1.27)
-				)
-			)
-		)
-		(property "Sim.Type" "VDMOS"
-			(at 158.75 87.63 0)
-			(hide yes)
-			(show_name no)
-			(do_not_autoplace no)
-			(effects
-				(font
-					(size 1.27 1.27)
-				)
-			)
-		)
-		(property "Sim.Pins" "1=D 2=G 3=S"
-			(at 158.75 91.44 0)
-			(hide yes)
-			(show_name no)
-			(do_not_autoplace no)
-			(effects
-				(font
-					(size 1.27 1.27)
-				)
-			)
-		)
-		(pin "2"
-		)
-		(pin "1"
-		)
-		(pin "3"
-		)
-		(instances
-			(project "Pack_Controller"
-				(path "/58a1c93e-baba-4d23-9191-955e00968735/bb6d2c27-83db-4480-8c62-fedc9a39072f"
-					(reference "Q2303")
-					(unit 1)
-				)
-			)
-		)
-	)
-	(symbol
 		(lib_id "power:GND")
 		(at 191.77 55.88 0)
@@
 			)
 		)
-		(property "Value" "1.5MR"
+		(property "Value" "10kR"
 			(at 242.824 50.8 90)
 			(show_name no)
@@
 			)
 		)
-		(property "Footprint" "Capacitor_SMD:C_0603_1608Metric_Pad1.08x0.95mm_HandSolder"
+		(property "Footprint" "Capacitor_SMD:C_0805_2012Metric"
 			(at 89.2048 80.01 0)
 			(hide yes)
@@
 			)
 		)
-		(property "Value" "1.5MR"
+		(property "Value" "39kR"
 			(at 238.76 42.164 90)
 			(show_name no)
@@
 					(unit 1)
 				)
+			)
+		)
+	)
+	(symbol
+		(lib_id "Diode:BAT46")
+		(at 156.21 106.68 0)
+		(unit 1)
+		(body_style 1)
+		(exclude_from_sim no)
+		(in_bom yes)
+		(on_board yes)
+		(in_pos_files yes)
+		(dnp no)
+		(property "Reference" "D2303"
+			(at 156.21 104.394 0)
+			(show_name no)
+			(do_not_autoplace no)
+			(effects
+				(font
+					(size 1.27 1.27)
+				)
+			)
+		)
+		(property "Value" "BAT46"
+			(at 156.21 109.22 0)
+			(show_name no)
+			(do_not_autoplace no)
+			(effects
+				(font
+					(size 1.27 1.27)
+				)
+			)
+		)
+		(property "Footprint" "Diode_SMD:D_SOD-123"
+			(at 156.21 111.125 0)
+			(hide yes)
+			(show_name no)
+			(do_not_autoplace no)
+			(effects
+				(font
+					(size 1.27 1.27)
+				)
+			)
+		)
+		(property "Datasheet" "http://www.vishay.com/docs/85662/bat46.pdf"
+			(at 156.21 106.68 0)
+			(hide yes)
+			(show_name no)
+			(do_not_autoplace no)
+			(effects
+				(font
+					(size 1.27 1.27)
+				)
+			)
+		)
+		(property "Description" "100V 0.15A Small Signal Schottky Diode, DO-35"
+			(at 156.21 106.68 0)
+			(hide yes)
+			(show_name no)
+			(do_not_autoplace no)
+			(effects
+				(font
+					(size 1.27 1.27)
+				)
+			)
+		)
+		(pin "1"
+		)
+		(pin "2"
+		)
+		(instances
+			(project "Pack_Controller"
+				(path "/58a1c93e-baba-4d23-9191-955e00968735/bb6d2c27-83db-4480-8c62-fedc9a39072f"
+					(reference "D2303")
+					(unit 1)
+				)

Commit message: many fixes
Parts:
- removed U2302: SN74LVC2G14DBV, Package_TO_SOT_SMD:SOT-23-6, symbol 74xGxx:SN74LVC2G14DBV
- added U2303: SN74LVC2G17DCK, Package_TO_SOT_SMD:SOT-23-6, symbol EKartParts:SN74LVC2G17
Connections:
- net +3.3V: now also U2303.5 (V_{CC})
- net GND: now also U2303.2 (GND)
- net IMD_OK: now also U2303.3 (2A); no longer D2303.1 (K), U2301.6 (nCLR)
- net at C2301.2, D2302.2 (A), R2301.2: now also U2303.1 (1A)
- net at U2301.7 (nPRE): now also U2303.6 (1Y)
- new net: D2303.1 (K), U2301.6 (nCLR), U2303.4 (2Y)
- no-connect marks 0 -> 1
Other:
- moved on the sheet: C2301, D2302, R2301

Commit message: yes
Parts:
- C2301: value 10uF 0805 16V -> 10uF 0805 35V
Changed lines of the file:
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@@
 			)
 		)
-		(property "Value" "10uF 0805 16V"
+		(property "Value" "10uF 0805 35V"
 			(at 80.01 86.36 0)
 			(show_name no)
