File: BMS/ECAD/PackController/Pack_Controller.kicad_pcb (KiCad board)
At the start: 2 copper layers, 1004.2 x 624 mm, 357 parts, among them K1101 KT12-1A-40L-THT, K1901 KT12-1A-40L-THT, Q1001 FDN352AP, Q1002 BC846, Q1101 DMP4065S-7, Q1102 IXTA08N100D2HV, Q1103 BC846, Q1104 IRLML0100TR, Q1901 IXTA08N100D2HV, Q1902 IRLML0100TR, Q1903 BC846, Q1904 DMP4065S-7, Q201 DMP4065S-7, Q202 BC846, Q2301 BC846, Q2302 DMP4065S-7, Q2303 DMP4065S-7, Q401 DMP4065S-7, Q402 BC846, Q403 DMP4065S-7, Q404 BC846, Q801 2N7002, T301 HM2106NL, T302 HM2106NL, U1001 SN74LVC2G02, U1002 74LVC86AD, U1003 74LV08, U1004 74LVC1G32Q, U1005 SN74LVC1G74, U1006 CD4072BPW, U1007 SN74LVC2G14DBV, U1101 TCLT1004, U1102 TCLT1004, U1103 TEA1-0505HI, U1801 R-78E3.3-1.0, U1802 R-78E5.0-1.0, U1901 TCLT1004, U1902 TCLT1004, U1903 TEA1-0505HI, U2001 ADUM3190, U2002 TEA1-0505HI, U201 MCP130-270 ITT, U202 STWD100YNYWY, U203 SN74LVC1G74, U204 STM32G483VET6, U205 24LC256-I/SN, U2301 SN74LVC1G74, U2302 SN74LVC2G14DBV, U301 TLE9015 DQU, U401 ADCMP393ARZ, U501 MCP2562-E-SN, U601 MCP2562-E-SN, U901 ADCMP393ARZ, U902 ADUM3190, U903 TEA1-0505HI, U904 ADUM3190, U905 TEA1-0505HI, Y201 WE830055951

Commit message: many fixes
Parts:
- removed C1101, C1102, C906, C913: 100nF 0603 100V, Capacitor_SMD:C_0603_1608Metric_Pad1.08x0.95mm_HandSolder
- removed C2001, C2011, C2013, C902, C903, C904, C909, C910, C911: 1uC 0805 50V, Capacitor_SMD:C_0805_2012Metric
- removed C2009, C905, C912: 100n 0603 50V, Capacitor_SMD:C_0603_1608Metric
- removed C907, C908, C914, C915: 10uF 0805 50V, Capacitor_SMD:C_0805_2012Metric
- removed D1903, D1904: BY2000, Diode_THT:D_DO-201AE_P12.70mm_Horizontal
- removed JP201, JP202: Jumper_2_Open, Jumper:SolderJumper-2_P1.3mm_Open_RoundedPad1.0x1.5mm
- removed Q2303: DMP4065S-7, Package_TO_SOT_SMD:SOT-23-3
- removed R1111, R1115: 9.09M 0.1%, Resistor_SMD:R_0603_1608Metric_Pad0.98x0.95mm_HandSolder
- removed R1113, R2007, R2009, R905, R906, R913, R914: 10kR, Resistor_SMD:R_0603_1608Metric_Pad0.98x0.95mm_HandSolder
- removed R1114: 1M 0.1%, Resistor_SMD:R_0603_1608Metric_Pad0.98x0.95mm_HandSolder
- removed R2002, R907, R911: 4.7MR 2512 3kV 1%, Resistor_SMD:R_2512_6332Metric_Pad1.40x3.35mm_HandSolder
- removed R2003, R912, R916: 39kR 2512 500V 1%, Resistor_SMD:R_2512_6332Metric_Pad1.40x3.35mm_HandSolder
- removed U2001, U902, U904: ADUM3190, Package_SO:QSOP-16_3.9x4.9mm_P0.635mm
- removed U2302: SN74LVC2G14DBV, Package_TO_SOT_SMD:SOT-23-6
- removed U903, U905: TEA1-0505HI, Converter_DCDC:Converter_DCDC_TRACO_TEA1-xxxxHI_THT
- added C1107: 100nF 0603 100V, Capacitor_SMD:C_0603_1608Metric_Pad1.08x0.95mm_HandSolder, F.Cu at (170.5, 68.8)
- added C1108: 100nF 0603 100V, Capacitor_SMD:C_0603_1608Metric_Pad1.08x0.95mm_HandSolder, F.Cu at (172.3, 68.8)
- added C1109: 100nF 0603 100V, Capacitor_SMD:C_0603_1608Metric_Pad1.08x0.95mm_HandSolder, F.Cu at (174.0, 68.8)
- added C1907: 100nF 0603 100V, Capacitor_SMD:C_0603_1608Metric_Pad1.08x0.95mm_HandSolder, F.Cu at (64.0, 52.0)
- added C2002: 100nC 0603 50V, Capacitor_SMD:C_0603_1608Metric, F.Cu at (116.3, 122.8)
- added C2004: 100pC 0603 50V, Capacitor_SMD:C_0603_1608Metric, F.Cu at (116.3, 125.3)
- added C2006: 100nC 0603 50V, Capacitor_SMD:C_0603_1608Metric, F.Cu at (116.3, 127.8)
- added C2008: 100nC 0603 16V, Capacitor_SMD:C_0603_1608Metric, F.Cu at (116.3, 130.3)
- added C2010: 1uC 0805 50V, Capacitor_SMD:C_0805_2012Metric, F.Cu at (110.0, 137.7)
- added C2012: 1uC 0805 16V, Capacitor_SMD:C_0805_2012Metric, F.Cu at (110.0, 140.7)
- added C2014: 1nC 0603 16V, Capacitor_SMD:C_0603_1608Metric, F.Cu at (116.3, 132.8)
- added C2015: 100nF 0603 100V, Capacitor_SMD:C_0603_1608Metric_Pad1.08x0.95mm_HandSolder, F.Cu at (100.9, 137.5)
- added C2016: 1uF 0805 50V, Capacitor_SMD:C_0805_2012Metric, F.Cu at (110.0, 143.7)
- added C916: 100nF 0603 100V, Capacitor_SMD:C_0603_1608Metric_Pad1.08x0.95mm_HandSolder, F.Cu at (86.6, 122.8)
- added C917: 1uF 0805 50V, Capacitor_SMD:C_0805_2012Metric, F.Cu at (70.8, 144.1)
- added C918: 100pC 0603 50V, Capacitor_SMD:C_0603_1608Metric, F.Cu at (90.7, 122.8)
- added C919: 100nF 0603 100V, Capacitor_SMD:C_0603_1608Metric_Pad1.08x0.95mm_HandSolder, F.Cu at (86.6, 125.3)
- added C920: 1uC 0805 50V, Capacitor_SMD:C_0805_2012Metric, F.Cu at (70.8, 147.1)
- added C921: 100nC 0603 50V, Capacitor_SMD:C_0603_1608Metric, F.Cu at (90.7, 125.3)
- added C922: 10uF 0805 50V, Capacitor_SMD:C_0805_2012Metric, F.Cu at (70.8, 150.1)
- added C923: 10uF 0805 50V, Capacitor_SMD:C_0805_2012Metric, F.Cu at (70.8, 153.1)
- added C924: 100nC 0603 16V, Capacitor_SMD:C_0603_1608Metric, F.Cu at (90.7, 127.8)
- added C925: 1uC 0805 16V, Capacitor_SMD:C_0805_2012Metric, F.Cu at (70.8, 156.1)
- added C926: 100nC 0603 50V, Capacitor_SMD:C_0603_1608Metric, F.Cu at (90.7, 130.3)
- added C927: 1nC 0603 16V, Capacitor_SMD:C_0603_1608Metric, F.Cu at (90.7, 132.8)
- added C928: 100nF 0603 100V, Capacitor_SMD:C_0603_1608Metric_Pad1.08x0.95mm_HandSolder, F.Cu at (86.6, 127.8)
- added C929: 1uF 0805 50V, Capacitor_SMD:C_0805_2012Metric, F.Cu at (75.2, 144.1)
- added C930: 100pC 0603 50V, Capacitor_SMD:C_0603_1608Metric, F.Cu at (94.7, 122.8)
- added C931: 100nF 0603 100V, Capacitor_SMD:C_0603_1608Metric_Pad1.08x0.95mm_HandSolder, F.Cu at (86.6, 130.3)
- added C932: 1uC 0805 50V, Capacitor_SMD:C_0805_2012Metric, F.Cu at (75.2, 147.1)
- added C933: 100nC 0603 50V, Capacitor_SMD:C_0603_1608Metric, F.Cu at (94.7, 125.3)
- added C934: 10uF 0805 50V, Capacitor_SMD:C_0805_2012Metric, F.Cu at (75.2, 150.1)
- added C935: 10uF 0805 50V, Capacitor_SMD:C_0805_2012Metric, F.Cu at (75.2, 153.1)
- added C936: 100nC 0603 16V, Capacitor_SMD:C_0603_1608Metric, F.Cu at (94.7, 127.8)
- added C937: 1uC 0805 16V, Capacitor_SMD:C_0805_2012Metric, F.Cu at (75.2, 156.1)
- added C938: 100nC 0603 50V, Capacitor_SMD:C_0603_1608Metric, F.Cu at (94.7, 130.3)
- added C939: 1nC 0603 16V, Capacitor_SMD:C_0603_1608Metric, F.Cu at (94.7, 132.8)
- added D1002: BAT46, Diode_SMD:D_SOD-123, F.Cu at (11.0, 117.7)
- added D1003: BAT46, Diode_SMD:D_SOD-123, F.Cu at (11.0, 121.0)
- added D101: BAT46, Diode_SMD:D_SOD-123, F.Cu at (3.18, 117.7)
- added D1106: BAT46, Diode_SMD:D_SOD-123, F.Cu at (177.5, 68.0)
- added D1108: MM3Z10VT1G (10V), Diode_SMD:D_SOD-323_HandSoldering, F.Cu at (169.5, 41.0)
- added Q101: BC846, Package_TO_SOT_SMD:SOT-23, F.Cu at (2.71, 126.0)
- added Q102: DMP4065S-7, Package_TO_SOT_SMD:SOT-23-3, F.Cu at (2.83, 121.6)
- added R1006: 1kR, Resistor_SMD:R_0603_1608Metric, F.Cu at (15.8, 121.9)
- added R101: 10kR, Resistor_SMD:R_0603_1608Metric, F.Cu at (-1.75, 117.3)
- added R102: 1kR, Resistor_SMD:R_0603_1608Metric, F.Cu at (-1.75, 119.8)
- added R103: 10kR, Resistor_SMD:R_0603_1608Metric, F.Cu at (-1.75, 122.3)
- added R104: 10kR, Resistor_SMD:R_0603_1608Metric, F.Cu at (-1.75, 124.8)
- added R1116: 100kR 0603, Resistor_SMD:R_0603_1608Metric_Pad0.98x0.95mm_HandSolder, F.Cu at (175.5, 67.0)
- added R1909: 100kR 0603, Resistor_SMD:R_0603_1608Metric_Pad0.98x0.95mm_HandSolder, F.Cu at (56.2, 50.5)
- added R1910: 500R 0805, Resistor_SMD:R_0805_2012Metric_Pad1.20x1.40mm_HandSolder, F.Cu at (17.2, 131.6)
- added R2004: 4.7MR 2512 3kV 0,1%, Resistor_SMD:R_2512_6332Metric_Pad1.40x3.35mm_HandSolder, F.Cu at (103.3, 124.0)
- added R2005: 4.7MR 2512 3kV 0,1%, Resistor_SMD:R_2512_6332Metric_Pad1.40x3.35mm_HandSolder, F.Cu at (103.3, 128.9)
- added R2006: 26.1kR 2512 500V 0,1%, Resistor_SMD:R_2512_6332Metric_Pad1.40x3.35mm_HandSolder, F.Cu at (103.3, 133.8)
- added R2008: 1kR, Resistor_SMD:R_0603_1608Metric_Pad0.98x0.95mm_HandSolder, F.Cu at (100.9, 140.0)
- added R915: 100kR 0.1%, Resistor_SMD:R_0603_1608Metric_Pad0.98x0.95mm_HandSolder, F.Cu at (79.0, 64.4)
- added R917: 100kR 0.1%, Resistor_SMD:R_0603_1608Metric_Pad0.98x0.95mm_HandSolder, F.Cu at (79.0, 62.2)
- added R918: 909kR 0.1%, Resistor_SMD:R_0603_1608Metric_Pad0.98x0.95mm_HandSolder, F.Cu at (79.0, 65.9)
- added R919: 909kR 0.1%, Resistor_SMD:R_0603_1608Metric_Pad0.98x0.95mm_HandSolder, F.Cu at (79.0, 60.7)
- added R920: 10kR, Resistor_SMD:R_0603_1608Metric_Pad0.98x0.95mm_HandSolder, F.Cu at (79.0, 68.4)
- added R921: 4.7MR 2512 3kV 0,1%, Resistor_SMD:R_2512_6332Metric_Pad1.40x3.35mm_HandSolder, F.Cu at (64.0, 124.0)
- added R922: 4.7MR 2512 3kV 0,1%, Resistor_SMD:R_2512_6332Metric_Pad1.40x3.35mm_HandSolder, F.Cu at (64.0, 128.9)
- added R923: 26.1kR 2512 500V 0,1%, Resistor_SMD:R_2512_6332Metric_Pad1.40x3.35mm_HandSolder, F.Cu at (64.0, 133.8)
- added R924: 1kR, Resistor_SMD:R_0603_1608Metric_Pad0.98x0.95mm_HandSolder, F.Cu at (86.6, 132.8)
- added R925: 4.7MR 2512 3kV 0,1%, Resistor_SMD:R_2512_6332Metric_Pad1.40x3.35mm_HandSolder, F.Cu at (64.0, 138.7)
- added R926: 4.7MR 2512 3kV 0,1%, Resistor_SMD:R_2512_6332Metric_Pad1.40x3.35mm_HandSolder, F.Cu at (64.0, 143.6)
- added R927: 26.1kR 2512 500V 0,1%, Resistor_SMD:R_2512_6332Metric_Pad1.40x3.35mm_HandSolder, F.Cu at (64.0, 148.5)
- added R928: 1kR, Resistor_SMD:R_0603_1608Metric_Pad0.98x0.95mm_HandSolder, F.Cu at (86.6, 135.3)
- added U1008: SN74LVC2G14DBV, Package_TO_SOT_SMD:SOT-23-6, F.Cu at (16.4, 118.4)
- added U1104: SN74LVC2G14DBV, Package_TO_SOT_SMD:SOT-23-6, F.Cu at (172.2, 65.2)
- added U1904: SN74LVC2G14DBV, Package_TO_SOT_SMD:SOT-23-6, F.Cu at (65.5, 48.5)
- added U2003: AMC0311R, EKartParts:AMC0311R Wide-body SOIC (DWV), F.Cu at (111.1, 128.8)
- added U2004: LP5907MFX-3.3, Package_TO_SOT_SMD:SOT-23-5, F.Cu at (114.8, 138.6)
- added U2303: SN74LVC2G17DCK, Package_TO_SOT_SMD:SOT-23-6, F.Cu at (-1.18, 132.7)
- added U906: LP5907MFX-3.3, Package_TO_SOT_SMD:SOT-23-5, F.Cu at (93.1, 144.9)
- added U907: AMC0311R, EKartParts:AMC0311R Wide-body SOIC (DWV), F.Cu at (80.7, 149.9)
- added U908: TEA1-0505HI, Converter_DCDC:Converter_DCDC_TRACO_TEA1-xxxxHI_THT, F.Cu at (74.8, 124.7)
- added U909: LP5907MFX-3.3, Package_TO_SOT_SMD:SOT-23-5, F.Cu at (93.1, 149.6)
- added U910: AMC0311R, EKartParts:AMC0311R Wide-body SOIC (DWV), F.Cu at (87.2, 149.9)
- added U911: TEA1-0505HI, Converter_DCDC:Converter_DCDC_TRACO_TEA1-xxxxHI_THT, F.Cu at (82.7, 124.7)
- C2301: footprint Capacitor_SMD:C_0603_1608Metric_Pad1.08x0.95mm_HandSolder -> Capacitor_SMD:C_0805_2012Metric
- D1901: value BY2000 -> BAT46; footprint Diode_THT:D_DO-201AE_P12.70mm_Horizontal -> Diode_SMD:D_SOD-123
- D1902: value BY2000 -> MM3Z10VT1G (10V); footprint Diode_THT:D_DO-201AE_P12.70mm_Horizontal -> Diode_SMD:D_SOD-323_HandSoldering
- Q1902: value IRLML0100TR -> IPD95R750P7; footprint Package_TO_SOT_SMD:SOT-23-3 -> Package_TO_SOT_SMD:TO-252-2
- R1105, R1901: footprint Resistor_SMD:R_0603_1608Metric_Pad0.98x0.95mm_HandSolder -> Resistor_SMD:R_1206_3216Metric
- R1106, R1902: value 10kR 0603 -> 100R 0603
- R1107, R1903: value 10kR 0603 -> 100kR 0603
- R1108, R1905: value 1kR 0805 0,25W -> 330R 0805 0,25W
- R1110: value 1M 0.1% -> 500R 0805; footprint Resistor_SMD:R_0603_1608Metric_Pad0.98x0.95mm_HandSolder -> Resistor_SMD:R_0805_2012Metric_Pad1.20x1.40mm_HandSolder
- R2001, R902, R904: value 4.7MR 2512 3kV 1% -> 500R 0805; footprint Resistor_SMD:R_2512_6332Metric_Pad1.40x3.35mm_HandSolder -> Resistor_SMD:R_0805_2012Metric_Pad1.20x1.40mm_HandSolder
- R901: value 68K 1% -> 68.1K 0.1%
- R903, R910: value 3.3k 1% -> 3.9k 0.1%
- R908: value 68K 1% -> 68,1K 0.1%
- U1007: value SN74LVC2G14DBV -> SN74LVC2G17DCK
- moved D2303 850.7 mm to (357.8, 43.3)
- moved U1007 807.6 mm to (315.5, 118.6)
- moved Q801 648.8 mm to (487.1, 72.7)
- moved R801 648.8 mm to (482.5, 71.8)
- moved R802 648.8 mm to (482.5, 74.3)
- moved R803 648.8 mm to (482.5, 76.8)
- moved R804 648.8 mm to (482.5, 79.3)
- moved R1001 630.9 mm to (311.1, 131.1)
- moved R1002 630.9 mm to (311.1, 133.7)
- moved R1003 630.9 mm to (311.1, 136.2)
- moved U1006 630.9 mm to (313.3, 126.6)
- moved U1004 622.2 mm to (306.0, 133.9)
- moved U1001 619.3 mm to (316.1, 131.8)
- moved U1005 619.3 mm to (316.1, 135.5)
- moved U1002 618.2 mm to (300.2, 118.1)
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Connections:
- net Net-(U1903--Vout) renamed /DCDC_AIR/TS_P_DCDC
- C1001 pad 1: Net-(U1005A-nPRE) -> Net-(U1007-1A)
- C1104 pad 1: Net-(U1103--Vout) -> /TS_P_VEHI
- C1105 pad 2: Net-(U1103--Vout) -> /TS_P_VEHI
- C1901 pad 1: Net-(Q1901-G) -> GND
- C1901 pad 2: Net-(Q1902-G) -> Net-(D1901-A)
- C1902 pad 1: Net-(Q1901-G) -> GND
- C1902 pad 2: Net-(Q1902-G) -> Net-(D1901-A)
- C2003 pad 2: +5V_VEHI -> +5V_DCDC
- C2005 pad 1: +5V_VEHI -> +5V_DCDC
- C2007 pad 2: Net-(U2002--Vin) -> GND
- C901 pad 1: Net-(U901E-VCC) -> +3.3V
- D1901 pad 1: Net-(D1901-K) -> /DCDC_AIR/DCDC_AIR_Enable
- D1902 pad 2: Net-(D1901-K) -> Net-(D1902-A)
- D2303 pad 1: /IMD_Monitoring/IMD_OK -> Net-(D2303-K)
- F1901 pad 2: Net-(D1901-A) -> Net-(Q1902-D)
- FAN101 pad 3: /MCU/FAN_PWM -> Net-(D101-K)
- HV_Indi101 pad 4: /TS_P_VEHI -> /TS_N_VEHI
- IMD_HV101 pad 4: /TS_P_VEHI -> /TS_N_VEHI
- K1901 pad 14: Net-(Q1901-G) -> Net-(D1902-A)
- Q1001 pad 3: /TSAL_GRN -> Net-(D1003-A)
- Q1901 pad 1: Net-(Q1901-G) -> Net-(D1902-A)
- Q1902 pad 1: Net-(D1902-K) -> Net-(Q1902-D)
- Q1902 pad 2: Net-(Q1902-G) -> Net-(D1902-K)
- Q1902 pad 3: Net-(Q1901-G) -> Net-(D1902-A)
- Q404 pad 1: /AIR/DANGER_V -> /AIR/DANGER_V_oD
- R1003 pad 2: /TSAL_Logik/GRN_ON -> /MCU/TSAL_GRN_ON
- R1004 pad 2: Net-(U1005A-nPRE) -> Net-(U1007-1A)
- R1110 pad 1: /HV_Measurement/V_ACCU -> /TS_P_VEHI
- R1110 pad 2: Net-(U901C--) -> /Precharge/+5V_TS_P_VEHI
- R1901 pad 2: Net-(Q1901-G) -> Net-(D1902-A)
- R1902 pad 1: Net-(Q1902-G) -> Net-(D1902-K)
- R1903 pad 2: Net-(Q1901-G) -> Net-(D1902-A)
- R1904 pad 1: Net-(D1904-K) -> /DCDC_AIR/+5V_TS_P_DCDC
- R2001 pad 1: /DCDC_AIR/TS_P_DCCD -> /TS_N_ACCU
- R2001 pad 2: Net-(R2001-Pad2) -> +5V_DCDC
- R408 pad 1: Net-(U401B-+) -> Net-(U401B--)
- R409 pad 1: /AIR/AIR_Error -> /AIR/nAIR_Error
- R410 pad 2: Net-(U401B-+) -> Net-(U401B--)
- R421 pad 1: /AIR/DANGER_V -> /AIR/DANGER_V_oD
- R902 pad 1: /TS_P_VEHI -> /TS_N_ACCU
- R902 pad 2: Net-(R902-Pad2) -> +5V_ACCU
- R904 pad 1: Net-(R902-Pad2) -> /TS_N_VEHI
- R904 pad 2: /TS_N_VEHI -> +5V_VEHI
- TH1901 pad 1: Net-(D1902-K) -> Net-(Q1902-D)
- U1001 pad 2: /AIR/AIR_Error -> /TSAL_Logik/AIR_Error
- U1003 pad 8: /TSAL_Logik/GRN_ON -> /MCU/TSAL_GRN_ON
- U1006 pad 12: /AIR/DANGER_V -> /TSAL_Logik/DANGER_V
- U1007 pad 4: Net-(U1007-1A) -> Net-(U1005A-nCLR)
- U1007 pad 6: Net-(U1005A-nCLR) -> Net-(U1005A-nPRE)
- U1101 pad 1: /Precharge/PCHRG_Enable -> Net-(U1104-1Y)
- U1103 pad 5: Net-(U1103--Vout) -> /TS_P_VEHI
- U1901 pad 1: /DCDC_AIR/DCDC_AIR_Enable -> Net-(U1904-1Y)
- U1901 pad 4: Net-(D1904-K) -> /DCDC_AIR/+5V_TS_P_DCDC
- U1902 pad 2: Net-(Q1901-G) -> Net-(D1902-A)
- U2002 pad 2: Net-(U2002--Vin) -> GND
- U2002 pad 7: +5V_VEHI -> +5V_DCDC
- U204 pad 36: Net-(JP201-A) -> +3.3V
- U204 pad 94: /AIR/AIR_Error -> /MCU/nAIR_Error
- U2301 pad 6: /IMD_Monitoring/IMD_OK -> Net-(D2303-K)
- U401 pad 1: /AIR/AIR_Error -> /AIR/nAIR_Error
- U401 pad 10: /AIR/AIR_N_AUX1 -> Net-(U401B--)
- U401 pad 11: Net-(U401B-+) -> /AIR/AIR_N_AUX1
- U401 pad 13: /AIR/AIR_Error -> /AIR/nAIR_Error
- U401 pad 6: /AIR/AIR_P_AUX1 -> Net-(U401B--)
- U401 pad 7: Net-(U401B-+) -> /AIR/AIR_P_AUX1
- U901 pad 1: /AIR/DANGER_V -> /HV_Measurement/DANGER_V_oD
- U901 pad 13: /MCU/nPRCHG_DONE -> /HV_Measurement/nPRCHG_DONE
- U901 pad 14: /AIR/DANGER_V -> /HV_Measurement/PRCHG_DONE
- U901 pad 3: Net-(U901E-VCC) -> +3.3V
Other:
- board size 1004.2 x 624 mm -> 280 x 80 mm

Commit message: add rule areas for hv separation
Parts:
- added C101: 10uF 1206 25V, Capacitor_SMD:C_1206_3216Metric, F.Cu at (151.8, 172.7)
- added C102: 47uF 25V, Capacitor_THT:CP_Radial_D6.3mm_P2.50mm, F.Cu at (143.8, 174.9)
- added D102: Z 12V (MM3Z12VT1G), Diode_SMD:D_SOD-323_HandSoldering, F.Cu at (151.6, 175.8)
- added D103: SMAJ15CA, Diode_SMD:D_SMA, F.Cu at (145.1, 181.1)
- added Q104: DMP4065S-7, Package_TO_SOT_SMD:SOT-23-3, F.Cu at (151.7, 181.1)
- added R105: 10kR, Resistor_SMD:R_0603_1608Metric, F.Cu at (151.1, 184.6)
- C1903, C1904, C1905, C1906, C2002, C2003, C2004, C2005, C2006, C2007, C2008, C2010, C2012, C2014, C2015, C2016, C916, C917, C918, C919, C920, C921, C922, C923, C924, C925, C926, C927, C928, C929, C930, C931, C932, C933, C934, C935, C936, C937, C938, C939, D1902, D1905, D1906, R1902, R1903, R1904, R2008, R921, R924, R928, U1901, U1902, U2003, U2004, U906, U907, U909, U910: moved to B.Cu
- C208: value 100nF 0603 6.3V -> 100nF 0603 16V
- R1110: value 500R 0805 -> 270R 0805
- R1910, R2001, R902, R904: value 500R 0805 -> 270R 0805; moved to B.Cu
- moved D1001 322.3 mm to (0.71, 182.0)
- moved C1006 318.0 mm to (-8.22, 194.1)
- moved D2301 317.3 mm to (71.8, 174.0)
- moved D2302 317.3 mm to (71.8, 177.4)
- moved D2303 317.3 mm to (71.8, 180.7)
- moved Q2301 317.3 mm to (71.3, 189.3)
- moved Q2302 317.3 mm to (76.6, 184.6)
- moved U2301 317.3 mm to (76.6, 189.0)
- moved C2301 317.3 mm to (76.0, 192.2)
- moved C2302 317.3 mm to (70.9, 192.7)
- moved R2301 317.3 mm to (66.7, 173.6)
- moved R2302 317.3 mm to (66.7, 176.1)
- moved R2303 317.3 mm to (66.7, 178.6)
- moved R2304 317.3 mm to (66.7, 181.2)
- moved R2305 317.3 mm to (66.7, 183.7)
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Connections:
- HV_DCDC101 pad 1: /DCDC_AIR/TS_P_DCCD -> /DCDC_AIR/TS_P_DCDC
- K1901 pad 13: /DCDC_AIR/TS_P_DCCD -> /DCDC_AIR/TS_P_DCDC
- MAIN_LV101 pad 2: +BATT -> /+Batt_In
- MAIN_LV101 pad 3: +BATT -> /+Batt_In
- R2004 pad 1: /DCDC_AIR/TS_P_DCCD -> /DCDC_AIR/TS_P_DCDC
- U1004 pad 1: /AIR/AIR_P_Actual -> /Precharge/PCHRG_Intended
- U1008 pad 1: /TSAL_Logik/nAIR_Error -> /AIR/nAIR_Error
- U1101 pad 1: Net-(U1104-1Y) -> /Precharge/PCHRG_Intended
- U1104 pad 6: Net-(U1104-1Y) -> /Precharge/PCHRG_Intended
- U204 pad 83: /MCU/nPRCHG_DONE -> /HV_Measurement/nPRCHG_DONE
- U204 pad 94: /MCU/nAIR_Error -> /AIR/nAIR_Error
- U901 pad 1: /HV_Measurement/DANGER_V_oD -> /AIR/DANGER_V_oD
- U901 pad 14: /HV_Measurement/PRCHG_DONE -> /AIR/DANGER_V_oD
Routing:
- net /TS_N_ACCU: track 0.00 -> 28.6 mm
- net +5V_ACCU: track 0.00 -> 17.6 mm
- net +3.3V_ACCU: track 0.00 -> 14.2 mm
- net Net-(U907-INP): track 0.00 -> 2.36 mm

Commit message: route HV components
Parts:
- R1109, U1102: moved to B.Cu
- moved U1903 30.3 mm to (31.0, 46.6)
- moved C1905 30.0 mm to (33.5, 45.5)
- moved R1910 27.0 mm to (34.2, 34.0)
- moved C1903 26.8 mm to (34.2, 30.2)
- moved C1904 26.8 mm to (34.2, 32.0)
- moved R2004 18.8 mm to (13.0, 13.8)
- moved R921 14.6 mm to (95.5, 19.5)
- moved R2005 14.2 mm to (17.8, 20.2), turned to 0 degrees
- moved D1905 11.8 mm to (64.8, 50.2), turned to 0 degrees
- moved HV_DCDC101 11.5 mm to (32.8, 23.8), turned to 90 degrees
- moved U1901 10.5 mm to (47.0, 40.2)
- moved K1901 8.38 mm to (65.8, 32.2)
- moved C1901 8.38 mm to (62.9, 72.8)
- moved C1902 8.38 mm to (61.4, 72.8)
- moved C1907 8.38 mm to (59.9, 72.8)
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Connections:
- C1106 pad 2: Net-(U1103--Vin) -> GND
- C1905 pad 2: Net-(U1903--Vin) -> GND
- U1103 pad 2: Net-(U1103--Vin) -> GND
- U1903 pad 2: Net-(U1903--Vin) -> GND
Routing:
- net /TS_N_ACCU: track 28.6 -> 171.4 mm, vias 0 -> 2
- net /TS_N_VEHI: track 0.00 -> 65.6 mm, vias 0 -> 2
- net /TS_P_ACCU: track 0.00 -> 51.9 mm
- net /DCDC_AIR/TS_P_DCDC: track 0.00 -> 49.2 mm, vias 0 -> 1
- net /TS_P_VEHI: track 0.00 -> 40.3 mm
- net Net-(D1902-A): track 0.00 -> 37.9 mm
- net Net-(U910-INP): track 0.00 -> 33.6 mm, vias 0 -> 1
- net Net-(D1108-A): track 0.00 -> 32.8 mm
- net Net-(D1902-K): track 0.00 -> 30.7 mm, vias 0 -> 1
- net /DCDC_AIR/+5V_TS_P_DCDC: track 0.00 -> 29.7 mm, vias 0 -> 1
- net /Precharge/+5V_TS_P_VEHI: track 0.00 -> 29.1 mm
- net +3.3V_DCDC: track 0.00 -> 19.8 mm, vias 0 -> 3
- net Net-(R1106-Pad2): track 0.00 -> 17.1 mm, vias 0 -> 2
- net Net-(U907-INP): track 2.36 -> 19.1 mm, vias 0 -> 1
- net +3.3V_VEHI: track 0.00 -> 15.7 mm
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Other:
- copper layers 2 -> 4

Commit message: most of layout complete
Parts:
- added D1903: BY2000, Diode_THT:D_DO-201AE_P12.70mm_Horizontal, F.Cu at (50.9, 26.2)
- C1003, C1601, C1701, C1803, C1805, C1806, C1901, C1902, C1907, C201, C202, C203, C214, C2301, C2302, C501, C502, C601, C602, D101, D1901, D2301, D2302, D2303, D401, D403, D501, D502, D601, D602, Q101, Q102, Q1903, Q1904, Q2301, Q2302, Q401, Q402, Q403, Q404, Q801, R101, R102, R103, R104, R1602, R1603, R1605, R1702, R1703, R1705, R1801, R1802, R1905, R1906, R1907, R1908, R1909, R1911, R1912, R215, R2301, R2302, R2303, R2304, R2305, R2306, R2307, R2308, R2310, R401, R402, R406, R407, R411, R412, R413, R414, R415, R416, R417, R418, R419, R420, R421, R422, R501, R502, R503, R601, R602, R603, R801, R802, R803, R804, U1006, U1904, U205, U2301, U2303, U501, U601: moved to B.Cu
- moved Q801 448.2 mm to (39.5, 50.8), turned to 90 degrees
- moved BUZZ101 445.6 mm to (43.0, 47.8), turned to 180 degrees
- moved R802 441.7 mm to (41.8, 46.0), turned to 180 degrees
- moved R804 441.4 mm to (42.0, 51.2), turned to -90 degrees
- moved R803 439.7 mm to (43.5, 51.2), turned to -90 degrees
- moved R801 437.9 mm to (45.0, 52.0), turned to -90 degrees
- moved C1503 404.8 mm to (88.2, 136.5), turned to -90 degrees
- moved NTC5 404.3 mm to (79.5, 127.0), turned to -90 degrees
- moved C1502 402.4 mm to (90.7, 136.5), turned to -90 degrees
- moved C1501 399.9 mm to (93.2, 136.5), turned to -90 degrees
- moved C1401 397.5 mm to (95.8, 136.5), turned to -90 degrees
- moved NTC4 396.3 mm to (87.3, 127.0), turned to -90 degrees
- moved C1301 395.0 mm to (98.3, 136.5), turned to -90 degrees
- moved D1503 392.4 mm to (101.0, 136.5), turned to -90 degrees
- moved Leak2 390.6 mm to (10.3, 47.8), turned to 90 degrees
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Connections:
- R1904 pad 1: /DCDC_AIR/+5V_TS_P_DCDC -> Net-(D1903-K)
- U1901 pad 4: /DCDC_AIR/+5V_TS_P_DCDC -> Net-(D1903-K)
Routing:
- net /AIR/SC_END: track 0.00 -> 201.7 mm, vias 0 -> 4
- net /MCU/PCHRG_ACTUAL: track 0.00 -> 193.2 mm, vias 0 -> 6
- net /Precharge/PCHRG_Intended: track 0.00 -> 183.3 mm, vias 0 -> 3
- net /MCU/ERRQ_Ioc_out: track 0.00 -> 182.2 mm, vias 0 -> 2
- net /MCU/ERRQ_ext_out: track 0.00 -> 181.8 mm, vias 0 -> 2
- net /MCU/ERRQ_ext: track 0.00 -> 180.8 mm, vias 0 -> 2
- net /MCU/ERRQ_res: track 0.00 -> 178.5 mm, vias 0 -> 2
- net /MCU/nSleep: track 0.00 -> 177.4 mm, vias 0 -> 2
- net /MCU/UART_HS_RX: track 0.00 -> 171.7 mm, vias 0 -> 2
- net /MCU/ERRQ: track 0.00 -> 168.4 mm, vias 0 -> 3
- net /MCU/UART_LS_RX: track 0.00 -> 165.9 mm, vias 0 -> 2
- net /MCU/UART_LS_TX: track 0.00 -> 151.4 mm, vias 0 -> 2
- net /MCU/UART_HS_TX: track 0.00 -> 149.2 mm, vias 0 -> 2
- net GND: track 0.00 -> 141.1 mm, vias 0 -> 31
- net /HV_Measurement/nDANGER_V: track 0.00 -> 111.0 mm, vias 0 -> 6
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Other:
- board size 280 x 80 mm -> 209.9 x 80 mm
- copper layers 4 -> 6

Commit message: yes
Parts:
- removed Q1101, Q1904: DMP4065S-7, Package_TO_SOT_SMD:SOT-23-3
- removed R908: 68,1K 0.1%, Resistor_SMD:R_0603_1608Metric_Pad0.98x0.95mm_HandSolder
- removed R910: 3.9k 0.1%, Resistor_SMD:R_0603_1608Metric_Pad0.98x0.95mm_HandSolder
- removed R915: 100kR 0.1%, Resistor_SMD:R_0603_1608Metric_Pad0.98x0.95mm_HandSolder
- removed R918, R919: 909kR 0.1%, Resistor_SMD:R_0603_1608Metric_Pad0.98x0.95mm_HandSolder
- added D104: DESD5V0S1BA-7, Diode_SMD:D_SOD-323, B.Cu at (77.5, 74.5)
- added G*** (x3): LOGO, LOGO, F.Cu at (189.0, 14.0)
- added Q1105: FDN352AP, Package_TO_SOT_SMD:SOT-23, F.Cu at (161.2, 60.5)
- added Q1905: FDN352AP, Package_TO_SOT_SMD:SOT-23, B.Cu at (73.0, 44.8)
- added R905: 909kR 0.1%, Resistor_SMD:R_0603_1608Metric_Pad0.98x0.95mm_HandSolder, F.Cu at (100.0, 52.5)
- C1001, C1002: value 1uF 16V -> 1uF 100V; footprint Capacitor_SMD:C_0603_1608Metric -> Capacitor_SMD:C_0805_2012Metric
- C101: value 10uF 1206 25V -> 10uF 0805 35V; footprint Capacitor_SMD:C_1206_3216Metric -> Capacitor_SMD:C_0805_2012Metric
- C1103, C1906: value 10uF 0805 25V -> 10uF 0805 35V
- C1106, C1904, C1905, C2005, C2007, C922, C923, C934: value 10uF 0805 50V -> 10uF 0805 35V
- C1301, C1401, C1501, C1502, C1503, C303, D1301, D1401, D1501, D1502, D1503, R1301, R1302, R1401, R1402, R1501, R1502, R1503, R1504, R1505, R1506, R310, R311: moved to B.Cu
- C2301: value 10uF 0805 16V -> 10uF 0805 35V
- C304: value 330nF 16V -> 330nF 50V; footprint Capacitor_SMD:C_1206_3216Metric -> Capacitor_SMD:C_0805_2012Metric; moved to B.Cu
- C305, C306, C307, C308, C310, C311, C312: value 2.2nC 1000V -> 2.2nC 100V; footprint Capacitor_SMD:C_1206_3216Metric -> Capacitor_SMD:C_0603_1608Metric
- C309: footprint Capacitor_SMD:C_1206_3216Metric -> Capacitor_SMD:C_0603_1608Metric
- C313, C314, C315, C316: value 220pC 1000V -> 220pC 100V; footprint Capacitor_SMD:C_1206_3216Metric -> Capacitor_SMD:C_0603_1608Metric
- moved C1503 106.9 mm to (171.5, 69.5), turned to 0 degrees
- moved NTC5 104.7 mm to (170.4, 75.0), turned to 90 degrees
- moved C1502 98.7 mm to (163.5, 69.8), turned to 0 degrees
- moved D1503 91.8 mm to (167.8, 73.5), turned to 90 degrees
- moved C1501 91.4 mm to (155.8, 69.8), turned to 0 degrees
- moved NTC4 91.4 mm to (162.5, 75.0), turned to 90 degrees
- moved R1506 85.5 mm to (173.0, 72.5)
- moved D1502 84.7 mm to (160.2, 73.2), turned to 90 degrees
- moved C1401 84.4 mm to (147.8, 70.0), turned to 0 degrees
- moved R1505 81.0 mm to (173.0, 76.2), turned to 90 degrees
- moved NTC3 79.1 mm to (154.7, 75.0), turned to 90 degrees
- moved C1301 78.2 mm to (139.8, 70.2), turned to 0 degrees
- moved D1501 77.8 mm to (152.2, 73.2), turned to 90 degrees
- moved R1504 77.8 mm to (165.0, 72.2)
- moved R1503 73.3 mm to (165.0, 76.0), turned to 90 degrees
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Connections:
- C1301 pad 2: /TempMeas/NTC1/NTCSig -> /MCU/NTC1_Sig
- C1401 pad 2: /TempMeas/NTC2/NTCSig -> /MCU/NTC2_Sig
- C1501 pad 2: /TempMeas/NTC3/NTCSig -> /MCU/NTC3_Sig
- C1502 pad 2: /TempMeas/NTC4/NTCSig -> /MCU/NTC4_Sig
- C1503 pad 2: /TempMeas/NTC5/NTCSig -> /MCU/NTC5_Sig
- NTC1 pad 1: /TempMeas/NTC1_+ -> /TempMeas/NTC1/NTC+
- NTC1 pad 2: /TempMeas/NTC1_-_4 -> GND
- NTC2 pad 1: /TempMeas/NTC1_+_4 -> /TempMeas/NTC2/NTC+
- NTC2 pad 2: /TempMeas/NTC1_- -> GND
- NTC3 pad 1: /TempMeas/NTC1_+_3 -> /TempMeas/NTC3/NTC+
- NTC3 pad 2: /TempMeas/NTC1_-_1 -> GND
- NTC4 pad 1: /TempMeas/NTC1_+_2 -> /TempMeas/NTC4/NTC+
- NTC4 pad 2: /TempMeas/NTC1_-_2 -> GND
- NTC5 pad 1: /TempMeas/NTC1_+_1 -> /TempMeas/NTC5/NTC+
- NTC5 pad 2: /TempMeas/NTC1_-_3 -> GND
- R1302 pad 1: /TempMeas/NTC1/NTCSig -> /MCU/NTC1_Sig
- R1402 pad 1: /TempMeas/NTC2/NTCSig -> /MCU/NTC2_Sig
- R1502 pad 1: /TempMeas/NTC3/NTCSig -> /MCU/NTC3_Sig
- R1504 pad 1: /TempMeas/NTC4/NTCSig -> /MCU/NTC4_Sig
- R1506 pad 1: /TempMeas/NTC5/NTCSig -> /MCU/NTC5_Sig
- R901 pad 2: Net-(U901B--) -> Net-(U901A-+)
- R903 pad 1: Net-(U901B--) -> Net-(U901A-+)
- U901 pad 11: Net-(U901D-+) -> Net-(U901C--)
- U901 pad 6: Net-(U901B--) -> Net-(U901A-+)
Routing:
- net +3.3V: track 80.7 -> 809.2 mm, vias 2 -> 41
- net +5V: track 35.2 -> 306.8 mm, vias 0 -> 8
- net GND: track 141.1 -> 336.9 mm, vias 31 -> 152
- net +BATT: track 58.0 -> 246.5 mm, vias 0 -> 5
- net /MCU/NTC5_Sig: track 0.00 -> 149.7 mm, vias 0 -> 4
- net /MCU/NTC4_Sig: track 0.00 -> 127.9 mm, vias 0 -> 2
- net /MCU/NTC2_Sig: track 0.00 -> 126.6 mm, vias 0 -> 2
- net /MCU/NTC3_Sig: track 0.00 -> 126.5 mm, vias 0 -> 2
- net /MCU/NTC1_Sig: track 0.00 -> 126.0 mm, vias 0 -> 2
- net /MCU/ERRQ_Ioc_out: track 182.2 -> 140.9 mm, vias 2 -> 4
- net /MCU/ERRQ_ext_out: track 181.8 -> 141.5 mm, vias 2 -> 5
- net /MCU/ERRQ_res: track 178.5 -> 145.3 mm, vias 2 -> 4
- net /MCU/UART_LS_TX: track 151.4 -> 119.0 mm
- net /MCU/ERRQ: track 168.4 -> 136.5 mm
- net /MCU/ERRQ_ext: track 180.8 -> 149.7 mm, vias 2 -> 4
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- added copper zone on In1.Cu, net GND
- added copper zone on In2.Cu, net GND
- added copper zone on In3.Cu, net GND
- added copper zone on In4.Cu, net GND
Other:
- board size 209.9 x 80 mm -> 199.9 x 80 mm
- board text added: "1"
- board text added: "2"
- board text added: "3"
- board text added: "4"
- board text added: "5"
- board text added: "6"
- board text added: "Coat PCB before use!"
- board text added: "HV"
- board text added: "LV"
- board text added: "PackController V1.0 Q3 2026 Lukas D. Max. 800V"
- board text added: "Plastic Screw only"
