File: BMS/ECAD/PackController/Pack_Controller.kicad_sch (KiCad schematic)
At the start: 6 parts, among them J101 Conn_01x10

Commit message: Add several auxilary circuits to BMS Master
Parts:
- removed J101: Conn_01x10, symbol Connector_Generic:Conn_01x10
- added FAN: (no value), Connector_Molex:Molex_Micro-Fit_3.0_43650-0315_1x03_P3.00mm_Vertical, symbol Connector_Generic:Conn_01x03
- added HV_DCDC, IMD_HV: 436500415, Connector_Molex:Molex_Micro-Fit_3.0_43650-0415_1x04_P3.00mm_Vertical, symbol Connector_Generic:Conn_01x04
- added IMD_LV: (no value), Connector_Molex:Molex_Micro-Fit_3.0_43045-0612_2x03_P3.00mm_Vertical, symbol Connector_Generic:Conn_01x06
- added MAIN_LV: (no value), Connector_Molex:Molex_Micro-Fit_3.0_43045-1212_2x06_P3.00mm_Vertical, symbol Connector_Generic:Conn_01x12
- BUZZ: renamed from BUZZ101; value Conn_01x02 -> (none); footprint (none) -> Connector_Molex:Molex_Micro-Fit_3.0_43650-0215_1x02_P3.00mm_Vertical
- HV_ACCU, HV_VEHI: footprint Connector_PinSocket_1.00mm:PinSocket_1x04_P1.00mm_Vertical -> Connector_Molex:Molex_Micro-Fit_3.0_43650-0415_1x04_P3.00mm_Vertical
- ISOUART_H, ISOUART_L: footprint Connector_PinSocket_1.00mm:PinSocket_1x02_P1.00mm_Vertical -> Connector_Molex:Molex_Micro-Fit_3.0_43650-0215_1x02_P3.00mm_Vertical
Connections:
- net +BATT: now also FAN.2 (Pin_2), IMD_LV.2 (Pin_2), MAIN_LV.2 (Pin_2), MAIN_LV.3 (Pin_3)
- net CAN1/CAN_N: now also MAIN_LV.7 (Pin_7)
- net CAN1/CAN_P: now also MAIN_LV.6 (Pin_6)
- net CAN2/CAN_N: now also MAIN_LV.9 (Pin_9)
- net CAN2/CAN_P: now also MAIN_LV.8 (Pin_8)
- net GND: now also FAN.1 (Pin_1), IMD_LV.1 (Pin_1), IMD_LV.3 (Pin_3), MAIN_LV.4 (Pin_4), MAIN_LV.5 (Pin_5)
- net HV_Measurement/TS_N_ACCU renamed TS_N_ACCU
- net HV_Measurement/TS_N_VEHI renamed TS_N_VEHI
- net HV_Measurement/TS_P_ACCU renamed TS_P_ACCU
- net HV_Measurement/TS_P_VEHI renamed TS_P_VEHI
- net TS_P_VEHI: now also IMD_HV.1 (Pin_1), IMD_HV.4 (Pin_4)
- new net DCDC_AIR/TS_P_DCCD: HV_DCDC.1 (Pin_1)
- new net GND Hoop: IMD_LV.4 (Pin_4), MAIN_LV.11 (Pin_11)
- new net HV_Measurement_DCDC/TS_N_ACCU: HV_DCDC.4 (Pin_4)
- new net IMD_Monitoring/M_HSLS: IMD_LV.5 (Pin_5)
- new net IMD_Monitoring/OK_HS: IMD_LV.6 (Pin_6)
- new net IMD_Monitoring/SC_In: MAIN_LV.1 (Pin_1)
- new net MCU/FAN_PWM: FAN.3 (Pin_3)
- new net TSAL_GRN: MAIN_LV.10 (Pin_10)
- no-connect marks 4 -> 8
Other:
- added sheet DCDC_AIR (DCDC_AIR.kicad_sch)
- added sheet HV_Measurement_DCDC (HV_Measurement_DCDC.kicad_sch)
- added sheet IMD_Monitoring (IMD_Monitoring.kicad_sch)
- sheet MCU ports: added DCDC_AIR_ACTUAL, DCDC_AIR_SWITCH, FAN_PWM, IMD_OK, IMD_SC_Closed, IMD_State, NTC4_Sig, NTC5_Sig, V_DCDC; removed none
- sheet TSAL_Logik ports: added AIR_Error, AIR_N_Actual, AIR_N_Intended, AIR_P_Actual, AIR_P_Intended, DANGER_V, GRN_ON, PCHRG_ACTUAL, nDANGER_V; removed TSAL_GRN_ON
- moved on the sheet: BUZZ, HV_ACCU, HV_VEHI, ISOUART_H, ISOUART_L

Commit message: finalised schematic of pack controller
Parts:
- added HV_Indi101: 436500415, Connector_Molex:Molex_Micro-Fit_3.0_43650-0415_1x04_P3.00mm_Vertical, symbol Connector_Generic:Conn_01x04
- renumbered BUZZ to BUZZ101, FAN to FAN101, HV_ACCU to HV_ACCU101, HV_DCDC to HV_DCDC101, HV_VEHI to HV_VEHI101, IMD_HV to IMD_HV101, IMD_LV to IMD_LV101, ISOUART_H to ISOUART_H101, ISOUART_L to ISOUART_L101, MAIN_LV to MAIN_LV101
Connections:
- net TS_P_VEHI: now also HV_Indi101.1 (Pin_1), HV_Indi101.4 (Pin_4)
- no-connect marks 8 -> 10
Changed lines of the file:
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@@
+	)
+	(junction
+		(at 55.88 119.38)
+		(diameter 0)
+		(color 0 0 0 0)
 	)
 	(junction
@@
 	)
 	(junction
+		(at 58.42 127)
+		(diameter 0)
+		(color 0 0 0 0)
+	)
+	(junction
 		(at 133.35 147.32)
 		(diameter 0)
@@
 	)
 	(no_connect
+		(at 41.91 137.16)
+	)
+	(no_connect
 		(at 41.91 121.92)
 	)
@@
 	)
 	(no_connect
+		(at 41.91 134.62)
+	)
+	(no_connect
 		(at 41.91 124.46)
 	)
@@
 	(wire
 		(pts
+			(xy 55.88 119.38) (xy 55.88 132.08)
+		)
+		(stroke
+			(width 0)
+			(type default)
+		)
+	)
+	(wire
+		(pts
 			(xy 292.1 124.46) (xy 292.1 121.92)
 		)
@@
 	(wire
 		(pts
+			(xy 58.42 127) (xy 58.42 139.7)
+		)
+		(stroke
+			(width 0)
+			(type default)
+		)
+	)
+	(wire
+		(pts
 			(xy 271.78 124.46) (xy 292.1 124.46)
 		)
@@
 	(wire
 		(pts
+			(xy 41.91 139.7) (xy 58.42 139.7)
+		)
+		(stroke
+			(width 0)
+			(type default)
+		)
+	)
+	(wire
+		(pts
 			(xy 66.04 88.9) (xy 78.74 88.9)
 		)
@@
 		(pts
 			(xy 110.49 151.13) (xy 140.97 151.13)
+		)
+		(stroke
+			(width 0)
+			(type default)
+		)
+	)
+	(wire
+		(pts
+			(xy 41.91 132.08) (xy 55.88 132.08)
 		)
 		(stroke
@@
 		(in_pos_files yes)
 		(dnp no)
-		(property "Reference" "HV_ACCU"
+		(property "Reference" "HV_ACCU101"
 			(at 28.956 91.186 0)
 			(show_name no)
@@
 			(project "Pack_Controller"
 				(path "/58a1c93e-baba-4d23-9191-955e00968735"
-					(reference "HV_ACCU")
+					(reference "HV_ACCU101")
 					(unit 1)
 				)
@@
 		(in_pos_files yes)
 		(dnp no)
-		(property "Reference" "IMD_LV"
-			(at 307.594 91.44 0)
+		(property "Reference" "IMD_LV101"
+			(at 309.372 98.044 90)
 			(show_name no)
 			(do_not_autoplace no)
@@
 			(project "Pack_Controller"
 				(path "/58a1c93e-baba-4d23-9191-955e00968735"
-					(reference "IMD_LV")
+					(reference "IMD_LV101")
 					(unit 1)
 				)
@@
 		(in_pos_files yes)
 		(dnp no)
-		(property "Reference" "ISOUART_L"
-			(at 129.54 218.44 0)
+		(property "Reference" "ISOUART_L101"
+			(at 127.254 218.186 0)
 			(show_name no)
 			(do_not_autoplace no)
@@
 		)
 		(property "Value" "436500227"
-			(at 129.54 215.9 0)
+			(at 127.254 215.646 0)
 			(show_name no)
 			(do_not_autoplace no)
@@
 			(project "Pack_Controller"
 				(path "/58a1c93e-baba-4d23-9191-955e00968735"
-					(reference "ISOUART_L")
+					(reference "ISOUART_L101")
 					(unit 1)
 				)
@@
 		(dnp no)
 		(fields_autoplaced yes)
-		(property "Reference" "MAIN_LV"
+		(property "Reference" "MAIN_LV101"
 			(at 325.12 116.8399 0)
 			(show_name no)
@@
 			(project "Pack_Controller"
 				(path "/58a1c93e-baba-4d23-9191-955e00968735"
-					(reference "MAIN_LV")
+					(reference "MAIN_LV101")
 					(unit 1)
 				)
@@
 		(in_pos_files yes)
 		(dnp no)
-		(property "Reference" "IMD_HV"
+		(property "Reference" "IMD_HV101"
 			(at 28.956 124.206 0)
 			(show_name no)
@@
 			(project "Pack_Controller"
 				(path "/58a1c93e-baba-4d23-9191-955e00968735"
-					(reference "IMD_HV")
+					(reference "IMD_HV101")
 					(unit 1)
 				)
@@
 		(in_pos_files yes)
 		(dnp no)
-		(property "Reference" "ISOUART_H"
-			(at 129.54 212.09 0)
+		(property "Reference" "ISOUART_H101"
+			(at 127.254 211.836 0)
 			(show_name no)
 			(do_not_autoplace no)
@@
 		)
 		(property "Value" "436500227"
-			(at 129.54 209.55 0)
+			(at 127.254 209.296 0)
 			(show_name no)
 			(do_not_autoplace no)
@@
 			(project "Pack_Controller"
 				(path "/58a1c93e-baba-4d23-9191-955e00968735"
-					(reference "ISOUART_H")
+					(reference "ISOUART_H101")
 					(unit 1)
 				)
@@
 		(in_pos_files yes)
 		(dnp no)
-		(fields_autoplaced yes)
-		(property "Reference" "FAN"
-			(at 247.65 71.1199 0)
+		(property "Reference" "FAN101"
+			(at 248.158 72.644 0)
 			(show_name no)
 			(do_not_autoplace no)
@@
 			(project "Pack_Controller"
 				(path "/58a1c93e-baba-4d23-9191-955e00968735"
-					(reference "FAN")
+					(reference "FAN101")
+					(unit 1)
+				)
+			)
+		)
+	)
+	(symbol
+		(lib_id "Connector_Generic:Conn_01x04")
+		(at 36.83 134.62 0)
+		(mirror y)
+		(unit 1)
+		(body_style 1)
+		(exclude_from_sim no)
+		(in_bom yes)
+		(on_board yes)
+		(in_pos_files yes)
+		(dnp no)
+		(property "Reference" "HV_Indi101"
+			(at 28.956 136.906 0)
+			(show_name no)
+			(do_not_autoplace no)
+			(effects
+				(font
+					(size 1.27 1.27)
+				)
+			)
+		)
+		(property "Value" "436500415"
+			(at 28.956 134.366 0)
+			(show_name no)
+			(do_not_autoplace no)
+			(effects
+				(font
+					(size 1.27 1.27)
+				)
+			)
+		)
+		(property "Footprint" "Connector_Molex:Molex_Micro-Fit_3.0_43650-0415_1x04_P3.00mm_Vertical"
+			(at 36.83 134.62 0)
+			(hide yes)
+			(show_name no)
+			(do_not_autoplace no)
+			(effects
+				(font
+					(size 1.27 1.27)
+				)
+			)
+		)
+		(property "Datasheet" ""
+			(at 36.83 134.62 0)
+			(hide yes)
+			(show_name no)
+			(do_not_autoplace no)
+			(effects
+				(font
+					(size 1.27 1.27)
+				)
+			)
+		)
+		(property "Description" "Generic connector, single row, 01x04, script generated (kicad-library-utils/schlib/autogen/connector/)"
+			(at 36.83 134.62 0)
+			(hide yes)
+			(show_name no)
+			(do_not_autoplace no)
+			(effects
+				(font
+					(size 1.27 1.27)
+				)
+			)
+		)
+		(pin "3"
+		)
+		(pin "4"
+		)
+		(pin "1"
+		)
+		(pin "2"
+		)
+		(instances
+			(project "Pack_Controller"
+				(path "/58a1c93e-baba-4d23-9191-955e00968735"
+					(reference "HV_Indi101")
 					(unit 1)
 				)
@@
 		(in_pos_files yes)
 		(dnp no)
-		(property "Reference" "BUZZ"
-			(at 287.528 139.7 0)
+		(property "Reference" "BUZZ101"
+			(at 290.068 139.446 0)
 			(show_name no)
 			(do_not_autoplace no)
@@
 			(project "Pack_Controller"
 				(path "/58a1c93e-baba-4d23-9191-955e00968735"
-					(reference "BUZZ")
+					(reference "BUZZ101")
 					(unit 1)
 				)
@@
 		(in_pos_files yes)
 		(dnp no)
-		(property "Reference" "HV_DCDC"
+		(property "Reference" "HV_DCDC101"
 			(at 114.3 61.722 0)
 			(show_name no)
@@
 			(project "Pack_Controller"
 				(path "/58a1c93e-baba-4d23-9191-955e00968735"
-					(reference "HV_DCDC")
+					(reference "HV_DCDC101")
 					(unit 1)
 				)
@@
 		(in_pos_files yes)
 		(dnp no)
-		(property "Reference" "HV_VEHI"
+		(property "Reference" "HV_VEHI101"
 			(at 28.956 102.616 0)
 			(show_name no)
@@
 			(project "Pack_Controller"
 				(path "/58a1c93e-baba-4d23-9191-955e00968735"
-					(reference "HV_VEHI")
+					(reference "HV_VEHI101")
 					(unit 1)
 				)

Commit message: many fixes
Parts:
- added D101: BAT46, Diode_SMD:D_SOD-123, symbol Diode:BAT46
- added Q101: BC846, Package_TO_SOT_SMD:SOT-23, symbol Transistor_BJT:BC846
- added Q102: DMP4065S-7, Package_TO_SOT_SMD:SOT-23-3, symbol Transistor_FET:Q_PMOS_GSD
- added R101, R103, R104: 10kR, Resistor_SMD:R_0603_1608Metric, symbol Device:R
- added R102: 1kR, Resistor_SMD:R_0603_1608Metric, symbol Device:R
Connections:
- net GND: now also Q101.2 (E), R101.2
- net MCU/FAN_PWM: now also R101.1, R102.2; no longer FAN101.3 (Pin_3)
- net TS_N_VEHI: now also HV_Indi101.4 (Pin_4), IMD_HV101.4 (Pin_4)
- net TS_P_VEHI: no longer HV_Indi101.4 (Pin_4), IMD_HV101.4 (Pin_4)
- new net: Q101.1 (B), R102.1
- new net: Q102.1 (G), R103.2, R104.1
- new net: D101.2 (A), Q102.3 (D)
- new net: D101.1 (K), FAN101.3 (Pin_3)
- new net: Q101.3 (C), R104.2
- new net +5V: Q102.2 (S), R103.1
Other:
- sheet MCU ports: added nAIR_Error; removed AIR_Error
- sheet TempMeas ports: added NTC4_Sig, NTC5_Sig; removed none
- moved on the sheet: FAN101

Commit message: add rule areas for hv separation
Parts:
- added C101: 10uF 1206 25V, Capacitor_SMD:C_1206_3216Metric, symbol Device:C
- added C102: 47uF 25V, Capacitor_THT:CP_Radial_D6.3mm_P2.50mm, symbol Device:C_Polarized
- added D102: Z 12V (MM3Z12VT1G), Diode_SMD:D_SOD-323_HandSoldering, symbol Device:D
- added D103: SMAJ15CA, Diode_SMD:D_SMA, symbol Device:D_TVS
- added Q104: DMP4065S-7, Package_TO_SOT_SMD:SOT-23-3, symbol Simulation_SPICE:PMOS
- added R105: 10kR, Resistor_SMD:R_0603_1608Metric, symbol Device:R
Connections:
- net HV_Measurement_DCDC/TS_N_ACCU is gone; now on net TS_N_ACCU: HV_DCDC101.4 (Pin_4)
- net +BATT: now also C101.2, C102.1, D102.1 (K), Q104.3 (S); no longer MAIN_LV101.2 (Pin_2), MAIN_LV101.3 (Pin_3)
- net GND: now also C101.1, C102.2, D103.1 (A1), R105.2
- net DCDC_AIR/TS_P_DCCD renamed DCDC_AIR/TS_P_DCDC
- new net: D102.2 (A), Q104.2 (G), R105.1
- new net +Batt_In: D103.2 (A2), MAIN_LV101.2 (Pin_2), MAIN_LV101.3 (Pin_3), Q104.1 (D)
Other:
- sheet AIR ports: added DANGER_V_oD, nAIR_Error; removed AIR_Error, DANGER_V
- sheet DCDC_AIR ports: added TS_P_DCDC; removed TS_P_DCCD, V_ACCU, V_DCDC
- sheet HV_Measurement ports: added DANGER_V_oD, PRCHG_DONE, nPRCHG_DONE; removed DANGER_V
- sheet Precharge ports: added PCHRG_Intended; removed PRCHG_DONE, V_ACCU, V_VEHI, nPRCHG_DONE
- sheet TSAL_Logik ports: added PCHRG_Intended, nAIR_Error; removed AIR_Error, DANGER_V
- moved on the sheet: HV_ACCU101, HV_DCDC101, HV_VEHI101, ISOUART_H101, ISOUART_L101

Commit message: most of layout complete
Other:
- moved on the sheet: ISOUART_H101
Changed lines of the file:
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@@
 	(wire
 		(pts
-			(xy 125.73 209.55) (xy 147.32 209.55)
+			(xy 106.68 209.55) (xy 147.32 209.55)
 		)
 		(stroke
@@
 	(wire
 		(pts
-			(xy 125.73 212.09) (xy 147.32 212.09)
+			(xy 106.68 212.09) (xy 147.32 212.09)
 		)
 		(stroke
@@
 			)
 			(justify left bottom)
+		)
+	)
+	(rule_area
+		(exclude_from_sim no)
+		(in_bom yes)
+		(on_board yes)
+		(dnp no)
+		(polyline
+			(pts
+				(xy 107.95 208.28) (xy 107.95 213.36) (xy 146.05 213.36) (xy 146.05 208.28)
+			)
+			(stroke
+				(width 0)
+				(type dash)
+			)
+			(fill
+				(type none)
+			)
+		)
+	)
+	(rule_area
+		(exclude_from_sim no)
+		(in_bom yes)
+		(on_board yes)
+		(dnp no)
+		(polyline
+			(pts
+				(xy 107.95 214.63) (xy 107.95 219.71) (xy 146.05 219.71) (xy 146.05 214.63)
+			)
+			(stroke
+				(width 0)
+				(type dash)
+			)
+			(fill
+				(type none)
+			)
+		)
+	)
+	(netclass_flag ""
+		(length 2.54)
+		(shape round)
+		(at 130.81 208.28 0)
+		(fields_autoplaced yes)
+		(effects
+			(font
+				(size 1.27 1.27)
+			)
+			(justify left bottom)
+		)
+		(property "Netzklasse" "HV800"
+			(at 131.5085 205.74 0)
+			(show_name no)
+			(do_not_autoplace no)
+			(effects
+				(font
+					(size 1.27 1.27)
+				)
+				(justify left)
+			)
+		)
+		(property "Component Class" ""
+			(at 34.29 11.43 0)
+			(show_name no)
+			(do_not_autoplace no)
+			(effects
+				(font
+					(size 1.27 1.27)
+					(italic yes)
+				)
+			)
 		)
 	)
@@
 		(length 2.54)
 		(shape round)
+		(at 110.49 219.71 180)
+		(fields_autoplaced yes)
+		(effects
+			(font
+				(size 1.27 1.27)
+			)
+			(justify right bottom)
+		)
+		(property "Netzklasse" "LOCAL_ISO_UART"
+			(at 111.1885 222.25 0)
+			(show_name no)
+			(do_not_autoplace no)
+			(effects
+				(font
+					(size 1.27 1.27)
+				)
+				(justify left)
+			)
+		)
+		(property "Component Class" ""
+			(at 13.97 22.86 0)
+			(show_name no)
+			(do_not_autoplace no)
+			(effects
+				(font
+					(size 1.27 1.27)
+					(italic yes)
+				)
+			)
+		)
+	)
+	(netclass_flag ""
+		(length 2.54)
+		(shape round)
+		(at 110.49 208.28 0)
+		(fields_autoplaced yes)
+		(effects
+			(font
+				(size 1.27 1.27)
+			)
+			(justify left bottom)
+		)
+		(property "Netzklasse" "LOCAL_ISO_UART"
+			(at 111.1885 205.74 0)
+			(show_name no)
+			(do_not_autoplace no)
+			(effects
+				(font
+					(size 1.27 1.27)
+				)
+				(justify left)
+			)
+		)
+		(property "Component Class" ""
+			(at 13.97 11.43 0)
+			(show_name no)
+			(do_not_autoplace no)
+			(effects
+				(font
+					(size 1.27 1.27)
+					(italic yes)
+				)
+			)
+		)
+	)
+	(netclass_flag ""
+		(length 2.54)
+		(shape round)
+		(at 130.81 219.71 180)
+		(fields_autoplaced yes)
+		(effects
+			(font
+				(size 1.27 1.27)
+			)
+			(justify right bottom)
+		)
+		(property "Netzklasse" "HV800"
+			(at 131.5085 222.25 0)
+			(show_name no)
+			(do_not_autoplace no)
+			(effects
+				(font
+					(size 1.27 1.27)
+				)
+				(justify left)
+			)
+		)
+		(property "Component Class" ""
+			(at 34.29 22.86 0)
+			(show_name no)
+			(do_not_autoplace no)
+			(effects
+				(font
+					(size 1.27 1.27)
+					(italic yes)
+				)
+			)
+		)
+	)
+	(netclass_flag ""
+		(length 2.54)
+		(shape round)
 		(at 48.26 88.9 0)
 		(fields_autoplaced yes)
@@
 		(property "Component Class" ""
 			(at 73.66 -21.59 0)
-			(show_name no)
-			(do_not_autoplace no)
-			(effects
-				(font
-					(size 1.27 1.27)
-					(italic yes)
-				)
-			)
-		)
-	)
-	(netclass_flag ""
-		(length 2.54)
-		(shape round)
-		(at 128.27 212.09 180)
-		(fields_autoplaced yes)
-		(effects
-			(font
-				(size 1.27 1.27)
-			)
-			(justify right bottom)
-		)
-		(property "Netzklasse" "HV800"
-			(at 128.9685 214.63 0)
-			(show_name no)
-			(do_not_autoplace no)
-			(effects
-				(font
-					(size 1.27 1.27)
-				)
-				(justify left)
-			)
-		)
-		(property "Component Class" ""
-			(at 105.41 133.35 0)
-			(show_name no)
-			(do_not_autoplace no)
-			(effects
-				(font
-					(size 1.27 1.27)
-					(italic yes)
-				)
-			)
-		)
-	)
-	(netclass_flag ""
-		(length 2.54)
-		(shape round)
-		(at 128.27 209.55 0)
-		(fields_autoplaced yes)
-		(effects
-			(font
-				(size 1.27 1.27)
-			)
-			(justify left bottom)
-		)
-		(property "Netzklasse" "HV800"
-			(at 128.9685 207.01 0)
-			(show_name no)
-			(do_not_autoplace no)
-			(effects
-				(font
-					(size 1.27 1.27)
-				)
-				(justify left)
-			)
-		)
-		(property "Component Class" ""
-			(at 105.41 130.81 0)
 			(show_name no)
 			(do_not_autoplace no)
@@
 	(symbol
 		(lib_id "Connector_Generic:Conn_01x02")
-		(at 120.65 209.55 0)
+		(at 101.6 209.55 0)
 		(mirror y)
 		(unit 1)
@@
 		(dnp no)
 		(property "Reference" "ISOUART_H101"
-			(at 110.744 211.836 0)
+			(at 91.694 211.836 0)
 			(show_name no)
 			(do_not_autoplace no)
@@
 		)
 		(property "Value" "436500227"
-			(at 110.744 209.296 0)
+			(at 91.694 209.296 0)
 			(show_name no)
 			(do_not_autoplace no)
@@
 		)
 		(property "Footprint" "Connector_Molex:Molex_Micro-Fit_3.0_43650-0215_1x02_P3.00mm_Vertical"
-			(at 120.65 209.55 0)
+			(at 101.6 209.55 0)
 			(hide yes)
 			(show_name no)
@@
 		)
 		(property "Datasheet" ""
-			(at 120.65 209.55 0)
+			(at 101.6 209.55 0)
 			(hide yes)
 			(show_name no)
@@
 		)
 		(property "Description" "Generic connector, single row, 01x02, script generated (kicad-library-utils/schlib/autogen/connector/)"
-			(at 120.65 209.55 0)
-			(hide yes)
-			(show_name no)
+			(at 101.6 209.55 0)
+			(hide yes)
+			(show_name no)

Commit message: yes
Parts:
- added D104: DESD5V0S1BA-7, Diode_SMD:D_SOD-323, symbol Device:D_TVS
- C101: value 10uF 1206 25V -> 10uF 0805 35V; footprint Capacitor_SMD:C_1206_3216Metric -> Capacitor_SMD:C_0805_2012Metric
Connections:
- net GND: now also D104.2 (A2)
- net IMD_Monitoring/SC_In: now also D104.1 (A1)
Changed lines of the file:
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@@
 	)
 	(junction
+		(at 314.96 97.79)
+		(diameter 0)
+		(color 0 0 0 0)
+	)
+	(junction
 		(at 355.6 77.47)
 		(diameter 0)
@@
 	(wire
 		(pts
+			(xy 327.66 97.79) (xy 327.66 100.33)
+		)
+		(stroke
+			(width 0)
+			(type default)
+		)
+	)
+	(wire
+		(pts
 			(xy 232.41 67.31) (xy 232.41 48.26)
 		)
@@
 	(wire
 		(pts
+			(xy 314.96 97.79) (xy 314.96 83.82)
+		)
+		(stroke
+			(width 0)
+			(type default)
+		)
+	)
+	(wire
+		(pts
 			(xy 349.25 87.63) (xy 349.25 88.9)
 		)
@@
 	(wire
 		(pts
-			(xy 314.96 104.14) (xy 314.96 83.82)
+			(xy 314.96 104.14) (xy 314.96 97.79)
 		)
 		(stroke
@@
 	(wire
 		(pts
+			(xy 323.85 97.79) (xy 327.66 97.79)
+		)
+		(stroke
+			(width 0)
+			(type default)
+		)
+	)
+	(wire
+		(pts
 			(xy 110.49 127) (xy 123.19 127)
 		)
@@
 	(wire
 		(pts
+			(xy 316.23 97.79) (xy 314.96 97.79)
+		)
+		(stroke
+			(width 0)
+			(type default)
+		)
+	)
+	(wire
+		(pts
 			(xy 109.22 52.07) (xy 110.49 52.07)
 		)
@@
 			(justify left bottom)
 		)
-		(property "Netzklasse" "HV800"
+		(property "Netclass" "HV800"
 			(at 131.5085 205.74 0)
 			(show_name no)
@@
 			(justify right bottom)
 		)
-		(property "Netzklasse" "HV0"
+		(property "Netclass" "HV0"
 			(at 48.9585 105.41 0)
 			(show_name no)
@@
 			(justify right bottom)
 		)
-		(property "Netzklasse" "LOCAL_ISO_UART"
+		(property "Netclass" "LOCAL_ISO_UART"
 			(at 111.1885 222.25 0)
 			(show_name no)
@@
 			(justify left bottom)
 		)
-		(property "Netzklasse" "LOCAL_ISO_UART"
+		(property "Netclass" "LOCAL_ISO_UART"
 			(at 111.1885 205.74 0)
 			(show_name no)
@@
 			(justify right bottom)
 		)
-		(property "Netzklasse" "HV800"
+		(property "Netclass" "HV800"
 			(at 131.5085 222.25 0)
 			(show_name no)
@@
 			(justify left bottom)
 		)
-		(property "Netzklasse" "HV800"
+		(property "Netclass" "HV800"
 			(at 48.9585 86.36 0)
 			(show_name no)
@@
 			(justify right bottom)
 		)
-		(property "Netzklasse" "HV0"
+		(property "Netclass" "HV0"
 			(at 48.9585 93.98 0)
 			(show_name no)
@@
 			(justify right bottom)
 		)
-		(property "Netzklasse" "HV800"
+		(property "Netclass" "HV800"
 			(at 97.2185 59.69 0)
 			(show_name no)
@@
 			(justify left bottom)
 		)
-		(property "Netzklasse" "HV800"
+		(property "Netclass" "HV800"
 			(at 48.9585 97.79 0)
 			(show_name no)
@@
 	)
 	(symbol
+		(lib_id "Device:D_TVS")
+		(at 320.04 97.79 0)
+		(unit 1)
+		(body_style 1)
+		(exclude_from_sim no)
+		(in_bom yes)
+		(on_board yes)
+		(in_pos_files yes)
+		(dnp no)
+		(property "Reference" "D104"
+			(at 320.04 100.33 0)
+			(show_name no)
+			(do_not_autoplace no)
+			(effects
+				(font
+					(size 1.27 1.27)
+				)
+			)
+		)
+		(property "Value" "DESD5V0S1BA-7"
+			(at 332.74 100.33 0)
+			(hide yes)
+			(show_name no)
+			(do_not_autoplace no)
+			(effects
+				(font
+					(size 1.27 1.27)
+				)
+			)
+		)
+		(property "Footprint" "Diode_SMD:D_SOD-323"
+			(at 320.04 97.79 0)
+			(hide yes)
+			(show_name no)
+			(do_not_autoplace no)
+			(effects
+				(font
+					(size 1.27 1.27)
+				)
+			)
+		)
+		(property "Datasheet" ""
+			(at 320.04 97.79 0)
+			(hide yes)
+			(show_name no)
+			(do_not_autoplace no)
+			(effects
+				(font
+					(size 1.27 1.27)
+				)
+			)
+		)
+		(property "Description" "Bidirectional transient-voltage-suppression diode"
+			(at 320.04 97.79 0)
+			(hide yes)
+			(show_name no)
+			(do_not_autoplace no)
+			(effects
+				(font
+					(size 1.27 1.27)
+				)
+			)
+		)
+		(pin "2"
+		)
+		(pin "1"
+		)
+		(instances
+			(project "Pack_Controller"
+				(path "/58a1c93e-baba-4d23-9191-955e00968735"
+					(reference "D104")
+					(unit 1)
+				)
+			)
+		)
+	)
+	(symbol
 		(lib_id "Device:C_Polarized")
 		(at 391.16 86.36 0)
@@
 			)
 		)
-		(property "Value" "10uF 1206 25V"
+		(property "Value" "10uF 0805 35V"
 			(at 386.588 78.486 90)
 			(show_name no)
@@
 			)
 		)
-		(property "Footprint" "Capacitor_SMD:C_1206_3216Metric"
+		(property "Footprint" "Capacitor_SMD:C_0805_2012Metric"
 			(at 380.0348 82.55 0)
 			(hide yes)
@@
 					(unit 1)
 				)
+			)
+		)
+	)
+	(symbol
+		(lib_id "power:GND")
+		(at 327.66 100.33 0)
+		(unit 1)
+		(body_style 1)
+		(exclude_from_sim no)
+		(in_bom yes)
+		(on_board yes)
+		(in_pos_files yes)
+		(dnp no)
+		(property "Reference" "#PWR0110"
+			(at 327.66 106.68 0)
+			(hide yes)
+			(show_name no)
+			(do_not_autoplace no)
+			(effects
+				(font
+					(size 1.27 1.27)
+				)
+			)
+		)
+		(property "Value" "GND"
+			(at 327.66 104.14 0)
+			(show_name no)
+			(do_not_autoplace no)
+			(effects
+				(font
+					(size 1.27 1.27)
+				)
+			)
+		)
+		(property "Footprint" ""
+			(at 327.66 100.33 0)
+			(hide yes)
+			(show_name no)
+			(do_not_autoplace no)
+			(effects
+				(font
+					(size 1.27 1.27)
+				)
+			)
+		)
+		(property "Datasheet" ""
+			(at 327.66 100.33 0)
+			(hide yes)
+			(show_name no)
+			(do_not_autoplace no)
+			(effects
+				(font
+					(size 1.27 1.27)
+				)
+			)
+		)
+		(property "Description" ""
+			(at 327.66 100.33 0)
+			(show_name no)
+			(do_not_autoplace no)
+			(effects
+				(font
+					(size 1.27 1.27)
+				)
+			)
+		)
+		(pin "1"
+		)
+		(instances
+			(project "Pack_Controller"
+				(path "/58a1c93e-baba-4d23-9191-955e00968735"
+					(reference "#PWR0110")
+					(unit 1)
+				)
