File: BMS/ECAD/PackController/TempMeas.kicad_sch (KiCad schematic)
At the start: 2 parts

Commit message: schematic finished, review tbd
Parts:
- removed Leak1, Leak2: Conn_01x02, symbol Connector_Generic:Conn_01x02
- added NTC1, NTC2, NTC3: Conn_01x02, symbol Connector_Generic:Conn_01x02
Connections:
- new net NTC1/NTC1_+: NTC1.1 (Pin_1)
- new net NTC1/NTC1_-: NTC1.2 (Pin_2)
- new net NTC2/NTC1_+: NTC2.1 (Pin_1)
- new net NTC2/NTC1_-: NTC2.2 (Pin_2)
- new net NTC3/NTC1_+: NTC3.1 (Pin_1)
- new net NTC3/NTC1_-: NTC3.2 (Pin_2)
Other:
- removed sheet LeakSens1
- removed sheet LeakSens2
- added sheet NTC1 (NTC1.kicad_sch)
- added sheet NTC2 (NTC1.kicad_sch)
- added sheet NTC3 (NTC1.kicad_sch)

Commit message: close to finish BMS master, only some footprints needed
Parts:
- renumbered NTC1 to NTC1201, NTC2 to NTC1202, NTC3 to NTC1203
Changed lines of the file:
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@@
 		(dnp no)
 		(fields_autoplaced yes)
-		(property "Reference" "NTC2"
+		(property "Reference" "NTC1202"
 			(at 158.75 90.1699 0)
 			(show_name no)
@@
 			(project "Pack_Controller"
 				(path "/58a1c93e-baba-4d23-9191-955e00968735/45830960-bd48-4e73-a3a7-091edb18d6d3"
-					(reference "NTC2")
+					(reference "NTC1202")
 					(unit 1)
 				)
@@
 		(dnp no)
 		(fields_autoplaced yes)
-		(property "Reference" "NTC3"
+		(property "Reference" "NTC1203"
 			(at 158.75 104.1399 0)
 			(show_name no)
@@
 			(project "Pack_Controller"
 				(path "/58a1c93e-baba-4d23-9191-955e00968735/45830960-bd48-4e73-a3a7-091edb18d6d3"
-					(reference "NTC3")
+					(reference "NTC1203")
 					(unit 1)
 				)
@@
 		(dnp no)
 		(fields_autoplaced yes)
-		(property "Reference" "NTC1"
+		(property "Reference" "NTC1201"
 			(at 158.75 76.1999 0)
 			(show_name no)
@@
 			(project "Pack_Controller"
 				(path "/58a1c93e-baba-4d23-9191-955e00968735/45830960-bd48-4e73-a3a7-091edb18d6d3"
-					(reference "NTC1")
+					(reference "NTC1201")
 					(unit 1)
 				)

Commit message: Add several auxilary circuits to BMS Master
Parts:
- added NTC4, NTC5: (no value), Connector_Molex:Molex_Micro-Fit_3.0_43650-0215_1x02_P3.00mm_Vertical, symbol Connector_Generic:Conn_01x02
- NTC1: renamed from NTC1201; value Conn_01x02 -> (none); footprint (none) -> Connector_Molex:Molex_Micro-Fit_3.0_43650-0215_1x02_P3.00mm_Vertical
- NTC2: renamed from NTC1202; value Conn_01x02 -> (none); footprint (none) -> Connector_Molex:Molex_Micro-Fit_3.0_43650-0215_1x02_P3.00mm_Vertical
- NTC3: renamed from NTC1203; value Conn_01x02 -> (none); footprint (none) -> Connector_Molex:Molex_Micro-Fit_3.0_43650-0215_1x02_P3.00mm_Vertical
Connections:
- new net NTC4/NTC1_+: NTC4.1 (Pin_1)
- new net NTC4/NTC1_-: NTC4.2 (Pin_2)
- new net NTC5/NTC1_+: NTC5.1 (Pin_1)
- new net NTC5/NTC1_-: NTC5.2 (Pin_2)
Other:
- added sheet NTC4 (NTC1.kicad_sch)
- added sheet NTC5 (NTC1.kicad_sch)

Commit message: yes
Connections:
- net NTC1/NTC1_+ renamed NTC1/NTC+
- net NTC1/NTC1_- renamed NTC1/NTC-
- net NTC2/NTC1_+ renamed NTC2/NTC+
- net NTC2/NTC1_- renamed NTC2/NTC-
- net NTC3/NTC1_+ renamed NTC3/NTC+
- net NTC3/NTC1_- renamed NTC3/NTC-
- net NTC4/NTC1_+ renamed NTC4/NTC+
- net NTC4/NTC1_- renamed NTC4/NTC-
- net NTC5/NTC1_+ renamed NTC5/NTC+
- net NTC5/NTC1_- renamed NTC5/NTC-
Other:
- sheet NTC1 ports: added NTC+, NTC-, NTCSig; removed NTC1_+, NTC1_-, NTC1_Sig
- sheet NTC2 ports: added NTC+, NTC-, NTCSig; removed NTC1_+, NTC1_-, NTC1_Sig
- sheet NTC3 ports: added NTC+, NTC-, NTCSig; removed NTC1_+, NTC1_-, NTC1_Sig
- sheet NTC4 ports: added NTC+, NTC-, NTCSig; removed NTC1_+, NTC1_-, NTC1_Sig
- sheet NTC5 ports: added NTC+, NTC-, NTCSig; removed NTC1_+, NTC1_-, NTC1_Sig
Changed lines of the file:
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@@
 			)
 		)
-		(pin "NTC1_+" input
+		(pin "NTCSig" input
+			(at 123.19 133.35 180)
+			(effects
+				(font
+					(size 1.27 1.27)
+				)
+				(justify left)
+			)
+		)
+		(pin "NTC-" input
+			(at 144.78 134.62 0)
+			(effects
+				(font
+					(size 1.27 1.27)
+				)
+				(justify right)
+			)
+		)
+		(pin "NTC+" input
 			(at 144.78 132.08 0)
-			(effects
-				(font
-					(size 1.27 1.27)
-				)
-				(justify right)
-			)
-		)
-		(pin "NTC1_Sig" input
-			(at 123.19 133.35 180)
-			(effects
-				(font
-					(size 1.27 1.27)
-				)
-				(justify left)
-			)
-		)
-		(pin "NTC1_-" input
-			(at 144.78 134.62 0)
 			(effects
 				(font
@@
 			)
 		)
-		(pin "NTC1_+" input
+		(pin "NTCSig" input
+			(at 123.19 119.38 180)
+			(effects
+				(font
+					(size 1.27 1.27)
+				)
+				(justify left)
+			)
+		)
+		(pin "NTC-" input
+			(at 144.78 120.65 0)
+			(effects
+				(font
+					(size 1.27 1.27)
+				)
+				(justify right)
+			)
+		)
+		(pin "NTC+" input
 			(at 144.78 118.11 0)
-			(effects
-				(font
-					(size 1.27 1.27)
-				)
-				(justify right)
-			)
-		)
-		(pin "NTC1_Sig" input
-			(at 123.19 119.38 180)
-			(effects
-				(font
-					(size 1.27 1.27)
-				)
-				(justify left)
-			)
-		)
-		(pin "NTC1_-" input
-			(at 144.78 120.65 0)
 			(effects
 				(font
@@
 			)
 		)
-		(pin "NTC1_+" input
+		(pin "NTCSig" input
+			(at 123.19 91.44 180)
+			(effects
+				(font
+					(size 1.27 1.27)
+				)
+				(justify left)
+			)
+		)
+		(pin "NTC-" input
+			(at 144.78 92.71 0)
+			(effects
+				(font
+					(size 1.27 1.27)
+				)
+				(justify right)
+			)
+		)
+		(pin "NTC+" input
 			(at 144.78 90.17 0)
-			(effects
-				(font
-					(size 1.27 1.27)
-				)
-				(justify right)
-			)
-		)
-		(pin "NTC1_Sig" input
-			(at 123.19 91.44 180)
-			(effects
-				(font
-					(size 1.27 1.27)
-				)
-				(justify left)
-			)
-		)
-		(pin "NTC1_-" input
-			(at 144.78 92.71 0)
 			(effects
 				(font
@@
 			)
 		)
-		(pin "NTC1_+" input
+		(pin "NTCSig" input
+			(at 123.19 105.41 180)
+			(effects
+				(font
+					(size 1.27 1.27)
+				)
+				(justify left)
+			)
+		)
+		(pin "NTC-" input
+			(at 144.78 106.68 0)
+			(effects
+				(font
+					(size 1.27 1.27)
+				)
+				(justify right)
+			)
+		)
+		(pin "NTC+" input
 			(at 144.78 104.14 0)
-			(effects
-				(font
-					(size 1.27 1.27)
-				)
-				(justify right)
-			)
-		)
-		(pin "NTC1_Sig" input
-			(at 123.19 105.41 180)
-			(effects
-				(font
-					(size 1.27 1.27)
-				)
-				(justify left)
-			)
-		)
-		(pin "NTC1_-" input
-			(at 144.78 106.68 0)
 			(effects
 				(font
@@
 			)
 		)
-		(pin "NTC1_+" input
+		(pin "NTCSig" input
+			(at 123.19 77.47 180)
+			(effects
+				(font
+					(size 1.27 1.27)
+				)
+				(justify left)
+			)
+		)
+		(pin "NTC+" input
 			(at 144.78 76.2 0)
 			(effects
@@
 			)
 		)
-		(pin "NTC1_Sig" input
-			(at 123.19 77.47 180)
-			(effects
-				(font
-					(size 1.27 1.27)
-				)
-				(justify left)
-			)
-		)
-		(pin "NTC1_-" input
+		(pin "NTC-" input
 			(at 144.78 78.74 0)
 			(effects
